File: 11_BUTTONS.kicad_sch (KiCad schematic)
At the start: 15 parts, among them SW1 BTN_LIGHT, SW2 BTN_UP, SW3 BTN_DOWN, SW4 BTN_START, SW5 BTN_BACK

Commit message: feat(kicad): assign and audit Rev-A footprints
Parts:
- SW1, SW2, SW3, SW4, SW5: footprint (none) -> Button_Switch_SMD:SW_SPST_EVQP7A
Changed lines of the file:
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@@
 			)
 		)
-		(property "Footprint" ""
+		(property "Footprint" "Button_Switch_SMD:SW_SPST_EVQP7A"
 			(at 110.49 92.71 0)
 			(hide yes)
@@
 			)
 		)
-		(property "Footprint" ""
+		(property "Footprint" "Button_Switch_SMD:SW_SPST_EVQP7A"
 			(at 110.49 113.03 0)
 			(hide yes)
@@
 			)
 		)
-		(property "Footprint" ""
+		(property "Footprint" "Button_Switch_SMD:SW_SPST_EVQP7A"
 			(at 110.49 157.48 0)
 			(hide yes)
@@
 			)
 		)
-		(property "Footprint" ""
+		(property "Footprint" "Button_Switch_SMD:SW_SPST_EVQP7A"
 			(at 110.49 134.62 0)
 			(hide yes)
@@
 			)
 		)
-		(property "Footprint" ""
+		(property "Footprint" "Button_Switch_SMD:SW_SPST_EVQP7A"
 			(at 110.49 73.66 0)
 			(hide yes)

Commit message: fix(pcba): resolve post-footprint freeze sanity items and freeze footprints
- Resolve Flatpak KICAD10_SYMBOL_DIR path discrepancy, reducing lib_symbol_issues to 0
- Re-audit Y1 and Y102 crystals against NDK NX1612SA; ground pads 2/4 for RF shield
- Reclassify SW1..SW5, J201, and J202 as Class C pending mechanical enclosure freeze
- Verify native ERC (0 errors), 83 interfaces (checked=83 mismatches=0), and 0 unintended net changes
- Add docs/project/post_footprint_freeze_sanity.md with FOOTPRINT FREEZE: PASS
Parts:
- SW1, SW2, SW3, SW4, SW5: footprint Button_Switch_SMD:SW_SPST_EVQP7A -> (none)
Changed lines of the file:
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@@
 			)
 		)
-		(property "Footprint" "Button_Switch_SMD:SW_SPST_EVQP7A"
+		(property "Footprint" ""
 			(at 110.49 92.71 0)
 			(hide yes)
@@
 			)
 		)
-		(property "Footprint" "Button_Switch_SMD:SW_SPST_EVQP7A"
+		(property "Footprint" ""
 			(at 110.49 113.03 0)
 			(hide yes)
@@
 			)
 		)
-		(property "Footprint" "Button_Switch_SMD:SW_SPST_EVQP7A"
+		(property "Footprint" ""
 			(at 110.49 157.48 0)
 			(hide yes)
@@
 			)
 		)
-		(property "Footprint" "Button_Switch_SMD:SW_SPST_EVQP7A"
+		(property "Footprint" ""
 			(at 110.49 134.62 0)
 			(hide yes)
@@
 			)
 		)
-		(property "Footprint" "Button_Switch_SMD:SW_SPST_EVQP7A"
+		(property "Footprint" ""
 			(at 110.49 73.66 0)
 			(hide yes)
