File: 11_BUTTONS.kicad_sch (KiCad schematic)
At the start: 0 parts

Commit message: updated schematics
Parts:
- added C1101, C1102, C1103, C1104, C1105: 47nF, Capacitor_SMD:C_0402_1005Metric, symbol Device:C
- added R1101, R1102, R1103, R1104, R1105: 100k, Resistor_SMD:R_0402_1005Metric, symbol Device:R
- added SW1: BTN_LIGHT, symbol Switch:SW_Push
- added SW2: BTN_UP, symbol Switch:SW_Push
- added SW3: BTN_DOWN, symbol Switch:SW_Push
- added SW4: BTN_START, symbol Switch:SW_Push
- added SW5: BTN_BACK, symbol Switch:SW_Push
Connections:
- new net BTN_BACK_N: C1105.1, R1105.2, SW5.1
- new net BTN_DOWN_N: C1103.1, R1103.2, SW3.1
- new net BTN_LIGHT_N: C1101.1, R1101.2, SW1.1
- new net BTN_START_N: C1104.1, R1104.2, SW4.1
- new net BTN_UP_N: C1102.1, R1102.2, SW2.1
- new net GND: C1101.2, C1102.2, C1103.2, C1104.2, C1105.2, SW1.2, SW2.2, SW3.2, SW4.2, SW5.2
- new net VOUT1_1V8: R1101.1, R1102.1, R1103.1, R1104.1, R1105.1
Other:
- note added: "100k + 47nF gives tau ~= 4.7ms (release threshold ~5.7ms for a 0.7*VDD GPIO VIH)."
- note added: "11_BUTTONS — FIVE PHYSICAL WATCH BUTTONS — ACTIVE LOW"
- note added: "Apollo510B GPIO input leakage is max 20nA, so 100k pull-ups retain very large DC noise margin."
- note added: "Do not rely on button labels as final GPIO ball assignments; those are frozen only during the Apollo integration pass."
- note added: "Each input has a 100k external pull-up to VOUT1_1V8 and 47nF hardware filter. Firmware should still debounce."
- note added: "Electrical behavior: unpressed = HIGH. Pressed = LOW. At 1.8V / 100k, a held button draws ~18uA."
- note added: "Final Apollo510B assignment: choose GPIOs valid in the selected low-power mode and configure falling-edge wake/interrupt."
- note added: "No exposed electrical button contacts are assumed. If the final mechanical design creates an external conductive ESD path, add local ESD protection after mechanical review."
- note added: "Switch footprints intentionally TBD until the exact sealed side-actuated tact switch / mechanical plunger stack is selected."
- title: (none) -> Rev-A — Physical buttons

Commit message: refactor(kicad): integrate Rev-A hierarchy and libraries
Changed lines of the file:
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@@
 		)
 	)
-	(label "VOUT1_1V8"
+	(hierarchical_label "VOUT1_1V8"
+		(shape passive)
 		(at 95.25 151.13 0)
 		(effects
@@
 		)
 	)
-	(label "BTN_BACK_N"
+	(hierarchical_label "BTN_BACK_N"
+		(shape output)
 		(at 90.17 162.56 180)
 		(effects
@@
 		)
 	)
-	(label "BTN_UP_N"
+	(hierarchical_label "BTN_UP_N"
+		(shape output)
 		(at 90.17 97.79 180)
 		(effects
@@
 		)
 	)
-	(label "BTN_START_N"
+	(hierarchical_label "BTN_START_N"
+		(shape output)
 		(at 90.17 139.7 180)
 		(effects
@@
 		)
 	)
-	(label "BTN_DOWN_N"
+	(hierarchical_label "BTN_DOWN_N"
+		(shape output)
 		(at 90.17 118.11 180)
 		(effects
@@
 		)
 	)
-	(label "BTN_LIGHT_N"
+	(hierarchical_label "BTN_LIGHT_N"
+		(shape output)
 		(at 90.17 78.74 180)
 		(effects

Commit message: foundation correction
Parts:
- C1101, C1102, C1103, C1104, C1105, R1101, R1102, R1103, R1104, R1105, SW1, SW2, SW3, SW4, SW5: Board (none) -> MAIN
Changed lines of the file:
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@@
 			)
 		)
-	)
+(property "Board" "MAIN" (at 0 0 0) (effects (font (size 1 1)) (hide yes)))
+)
 	(symbol
 		(lib_id "Device:C")
@@
 			)
 		)
-	)
+(property "Board" "MAIN" (at 0 0 0) (effects (font (size 1 1)) (hide yes)))
+)
 	(symbol
 		(lib_id "Switch:SW_Push")
@@
 			)
 		)
-	)
+(property "Board" "MAIN" (at 0 0 0) (effects (font (size 1 1)) (hide yes)))
+)
 	(symbol
 		(lib_id "power:GND")
@@
 			)
 		)
-	)
+(property "Board" "MAIN" (at 0 0 0) (effects (font (size 1 1)) (hide yes)))
+)
 	(symbol
 		(lib_id "Device:R")
@@
 			)
 		)
-	)
+(property "Board" "MAIN" (at 0 0 0) (effects (font (size 1 1)) (hide yes)))
+)
 	(symbol
 		(lib_id "Device:C")
@@
 			)
 		)
-	)
+(property "Board" "MAIN" (at 0 0 0) (effects (font (size 1 1)) (hide yes)))
+)
 	(symbol
 		(lib_id "power:GND")
@@
 			)
 		)
-	)
+(property "Board" "MAIN" (at 0 0 0) (effects (font (size 1 1)) (hide yes)))
+)
 	(symbol
 		(lib_id "Switch:SW_Push")
@@
 			)
 		)
-	)
+(property "Board" "MAIN" (at 0 0 0) (effects (font (size 1 1)) (hide yes)))
+)
 	(symbol
 		(lib_id "Device:R")
@@
 			)
 		)
-	)
+(property "Board" "MAIN" (at 0 0 0) (effects (font (size 1 1)) (hide yes)))
+)
 	(symbol
 		(lib_id "power:GND")
@@
 			)
 		)
-	)
+(property "Board" "MAIN" (at 0 0 0) (effects (font (size 1 1)) (hide yes)))
+)
 	(symbol
 		(lib_id "power:GND")
@@
 			)
 		)
-	)
+(property "Board" "MAIN" (at 0 0 0) (effects (font (size 1 1)) (hide yes)))
+)
 	(symbol
 		(lib_id "power:GND")
@@
 			)
 		)
-	)
+(property "Board" "MAIN" (at 0 0 0) (effects (font (size 1 1)) (hide yes)))
+)
 	(symbol
 		(lib_id "Device:R")
@@
 			)
 		)
-	)
+(property "Board" "MAIN" (at 0 0 0) (effects (font (size 1 1)) (hide yes)))
+)
 	(symbol
 		(lib_id "power:GND")
@@
 			)
 		)
-	)
+(property "Board" "MAIN" (at 0 0 0) (effects (font (size 1 1)) (hide yes)))
+)
 	(symbol
 		(lib_id "power:GND")
@@
 			)
 		)
-	)
+(property "Board" "MAIN" (at 0 0 0) (effects (font (size 1 1)) (hide yes)))
+)
 	(symbol
 		(lib_id "Device:C")
@@
 			)
 		)
-	)
+(property "Board" "MAIN" (at 0 0 0) (effects (font (size 1 1)) (hide yes)))
+)
 	(symbol
 		(lib_id "Switch:SW_Push")
@@
 			)
 		)
-	)
+(property "Board" "MAIN" (at 0 0 0) (effects (font (size 1 1)) (hide yes)))
+)
 	(symbol
 		(lib_id "power:GND")
@@
 			)
 		)
-	)
+(property "Board" "MAIN" (at 0 0 0) (effects (font (size 1 1)) (hide yes)))
+)
 	(symbol
 		(lib_id "Device:C")
@@
 			)
 		)
-	)
+(property "Board" "MAIN" (at 0 0 0) (effects (font (size 1 1)) (hide yes)))
+)
 	(symbol
 		(lib_id "Switch:SW_Push")
@@
 			)
 		)
-	)
+(property "Board" "MAIN" (at 0 0 0) (effects (font (size 1 1)) (hide yes)))
+)
 	(symbol
 		(lib_id "Device:R")
@@
 			)
 		)
-	)
+(property "Board" "MAIN" (at 0 0 0) (effects (font (size 1 1)) (hide yes)))
+)
 	(symbol
 		(lib_id "Switch:SW_Push")
@@
 			)
 		)
-	)
+(property "Board" "MAIN" (at 0 0 0) (effects (font (size 1 1)) (hide yes)))
+)
 	(symbol
 		(lib_id "Device:R")
@@
 			)
 		)
-	)
+(property "Board" "MAIN" (at 0 0 0) (effects (font (size 1 1)) (hide yes)))
+)
 	(symbol
 		(lib_id "power:GND")
@@
 			)
 		)
-	)
+(property "Board" "MAIN" (at 0 0 0) (effects (font (size 1 1)) (hide yes)))
+)
 	(symbol
 		(lib_id "Device:C")
@@
 			)
 		)
-	)
-)
+(property "Board" "MAIN" (at 0 0 0) (effects (font (size 1 1)) (hide yes)))
+)
+)
