File: 08_ENVIRONMENT.kicad_sch (KiCad schematic)
At the start: 0 parts

Commit message: updated schematics
Parts:
- added C801, C802, C803, C804: 100nF, Capacitor_SMD:C_0402_1005Metric, symbol Device:C
- added R801, R802: 4.7k, Resistor_SMD:R_0402_1005Metric, symbol Device:R
- added R803: 10k, Resistor_SMD:R_0402_1005Metric, symbol Device:R
- added U4: BMP585, LGA9_BMP585_BOS, symbol 2026-09-16_05-56-22:BMP585
- added U5: OPT4001DTSR, DTS0008A-MFG, symbol 2026-09-16_05-59-08:OPT4001DTSR
- added U6: MAX30208CLB+T, 21-100265_MXM, symbol 2026-09-16_05-57-26:MAX30208CLB+T
Connections:
- new net ALS_INT: R803.2, U5.7 (INT)
- new net BARO_INT: U4.5 (INT)
- new net ENV_I2C_SCL: R802.2, U4.1 (SCX), U5.5 (SCL), U6.9 (SCL)
- new net ENV_I2C_SDA: R801.2, U4.2 (SDX), U5.8 (SDA), U6.8 (SDA)
- new net GND: C801.2, C802.2, C803.2, C804.2, U4.3 (SDO), U4.6 (VSS), U5.2 (ADDR), U5.4 (GND), U6.10 (GPIO0), U6.4 (GND), U6.5 (GND), U6.6 (GND), U6.7 (GPIO1)
- new net VOUT1_1V8: C801.1, C802.1, C803.1, C804.1, R801.1, R802.1, R803.1, U4.4 (VDDIO), U4.7 (CSB), U4.8 (VDD), U5.1 (VDD), U6.1 (VDD), U6.2 (VDD), U6.3 (VDD)
- no-connect marks 0 -> 3
Other:
- note added: "08_ENVIRONMENT — BMP585 BAROMETER + MAX30208 SKIN TEMPERATURE + OPT4001 AMBIENT LIGHT — REV A"
- note added: "All three sensors use VOUT1_1V8. ENV_I2C_SDA/SCL are a 1.8 V I2C bus; Apollo pin assignment is deferred."
- note added: "BMP585 mechanical: pressure port must breathe through a hydrophobic/ePTFE vent; never cover the port with adhesive or conformal coating."
- note added: "BMP585: C803/C804 = 100nF at VDDIO/VDD. If either rail ramps faster than 10 us, Bosch recommends 10 ohm series limiting."
- note added: "BMP585: I2C mode; CSB=1.8 V, SDO=GND => 7-bit address 0x46; BARO_INT reserved for data-ready/interrupt."
- note added: "MAX30208 placement: skin-facing and thermally isolated from PMIC/SoC/PPG LEDs; thin traces/cutouts or flex improve skin tracking."
- note added: "MAX30208: GPIO1=GND and GPIO0=GND => fixed 7-bit address 0x50; temperature is polled, no interrupt pin consumed."
- note added: "OPT4001 mechanical: provide a real optical window / bezel opening; do not place behind opaque AMOLED or black mask."
- note added: "OPT4001DTSR: ADDR=GND => 0x44; ALS_INT is open-drain and uses R803=10k pull-up. C801=100nF at VDD."
- note added: "POWER / BUS PULL-UPS"
- note added: "R801/R802 = 4.7k pull-ups for provisional 400 kHz short sensor bus. Consolidate pull-ups if this bus is later shared with BMM350/PMIC."
- title: (none) -> Rev-A — Environmental sensors

Commit message: refactor(kicad): integrate Rev-A hierarchy and libraries
Parts:
- U4: footprint LGA9_BMP585_BOS -> sportwatch_custom:LGA9_BMP585_BOS
- U5: footprint DTS0008A-MFG -> sportwatch_custom:DTS0008A-MFG
- U6: footprint 21-100265_MXM -> sportwatch_custom:21-100265_MXM
Changed lines of the file:
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@@
 		)
 	)
-	(label "VOUT1_1V8"
+	(hierarchical_label "VOUT1_1V8"
+		(shape passive)
 		(at 205 32 0)
 		(effects
@@
 		)
 	)
-	(label "ENV_I2C_SCL"
+	(hierarchical_label "ENV_I2C_SCL"
+		(shape bidirectional)
 		(at 249 69.85 0)
 		(effects
@@
 		)
 	)
-	(label "ENV_I2C_SDA"
+	(hierarchical_label "ENV_I2C_SDA"
+		(shape bidirectional)
 		(at 48 73.66 180)
 		(effects
@@
 		)
 	)
-	(label "BARO_INT"
+	(hierarchical_label "BARO_INT"
+		(shape output)
 		(at 187 143.51 0)
 		(effects
@@
 		)
 	)
-	(label "ALS_INT"
+	(hierarchical_label "ALS_INT"
+		(shape output)
 		(at 235 50 0)
 		(effects
@@
 			)
 		)
-		(property "Footprint" "LGA9_BMP585_BOS"
+		(property "Footprint" "sportwatch_custom:LGA9_BMP585_BOS"
 			(at 132.08 133.35 0)
 			(hide yes)
@@
 			)
 		)
-		(property "Footprint" "DTS0008A-MFG"
+		(property "Footprint" "sportwatch_custom:DTS0008A-MFG"
 			(at 60.96 66.04 0)
 			(hide yes)
@@
 			)
 		)
-		(property "Footprint" "21-100265_MXM"
+		(property "Footprint" "sportwatch_custom:21-100265_MXM"
 			(at 196.85 67.31 0)
 			(hide yes)
