File: sportwatch_revA.kicad_sch (KiCad schematic)
At the start: 0 parts

Commit message: refactor(kicad): integrate Rev-A hierarchy and libraries
Other:
- sheet 01_APOLLO510B ports: added ALS_INT, APOLLO_BLE_ANT, APOLLO_BLE_AVDD_PA, APOLLO_RST_N, APOLLO_SWCLK, APOLLO_SWDIO, APOLLO_SWO_GPIO28, BARO_INT, BTN_BACK_N, BTN_DOWN_N, BTN_LIGHT_N, BTN_START_N, BTN_UP_N, DISP_QSPI_CLK, DISP_QSPI_CS, DISP_QSPI_IO0, DISP_QSPI_IO1, DISP_QSPI_IO2, DISP_QSPI_IO3, DISP_RST, DISP_TE, DISP_VCI_EN, EMMC_CLK, EMMC_CMD, EMMC_DAT0, EMMC_DAT1, EMMC_DAT2, EMMC_DAT3, EMMC_DAT4, EMMC_DAT5, EMMC_DAT6, EMMC_DAT7, EMMC_RST_N, ENV_I2C_SCL, ENV_I2C_SDA, GNSS_EXTINT, GNSS_TIMEPULSE, GNSS_UART_RX, GNSS_UART_TX, HAPTIC_I2C_SCL, HAPTIC_I2C_SDA, HAPTIC_NRST, HAPTIC_TRIG_INTZ, IMU_INT1, IMU_INT2, IMU_SPI_CS, IMU_SPI_MISO, IMU_SPI_MOSI, IMU_SPI_SCK, MAG_I2C_SCL, MAG_I2C_SDA, MAG_INT, PPG1_CS_N, PPG1_INT_N, PPG2_CS_N, PPG2_INT_N, PPG_SAMPLE_SYNC, PPG_SPI_MISO, PPG_SPI_MOSI, PPG_SPI_SCLK, SYS_3V3, TOUCH_INT, TOUCH_RST, TOUCH_SCL, TOUCH_SDA, VOUT1_1V8, WIFI_BUCKEN, WIFI_COEX_GRANT, WIFI_COEX_REQ, WIFI_COEX_STATUS, WIFI_HOST_IRQ, WIFI_IOVDD_EN, WIFI_QSPI_CLK, WIFI_QSPI_CS, WIFI_QSPI_IO0, WIFI_QSPI_IO1, WIFI_QSPI_IO2, WIFI_QSPI_IO3; removed none
- sheet 02_POWER ports: added MAG_I2C_SCL, MAG_I2C_SDA, SYS_3V3, VBAT, VOUT1_1V8, VOUT2_3V0_PROVISIONAL, VSYS; removed none
- sheet 03_DISPLAY ports: added DISP_QSPI_CLK, DISP_QSPI_CS, DISP_QSPI_IO0, DISP_QSPI_IO1, DISP_QSPI_IO2, DISP_QSPI_IO3, DISP_RST, DISP_TE, DISP_VCI_EN, SYS_3V3, TOUCH_INT, TOUCH_RST, TOUCH_SCL, TOUCH_SDA, VSYS; removed none
- sheet 04_PPG ports: added PPG1_CS_N, PPG1_INT_N, PPG2_CS_N, PPG2_INT_N, PPG_SAMPLE_SYNC, PPG_SPI_MISO, PPG_SPI_MOSI, PPG_SPI_SCLK, VOUT1_1V8; removed none
- sheet 05_GNSS ports: added GNSS_EXTINT, GNSS_RF, GNSS_TIMEPULSE, GNSS_UART_RX, GNSS_UART_TX, VOUT1_1V8, VOUT2_3V0_PROVISIONAL; removed none
- sheet 06_WIFI ports: added VBAT, VOUT1_1V8, WIFI_BUCKEN, WIFI_COEX_GRANT, WIFI_COEX_REQ, WIFI_COEX_STATUS, WIFI_HOST_IRQ, WIFI_IOVDD_EN, WIFI_QSPI_CLK, WIFI_QSPI_CS, WIFI_QSPI_IO0, WIFI_QSPI_IO1, WIFI_QSPI_IO2, WIFI_QSPI_IO3, WIFI_RF; removed none
- sheet 07_MOTION ports: added IMU_INT1, IMU_INT2, IMU_SPI_CS, IMU_SPI_MISO, IMU_SPI_MOSI, IMU_SPI_SCK, MAG_I2C_SCL, MAG_I2C_SDA, MAG_INT, VOUT1_1V8; removed none
- sheet 08_ENVIRONMENT ports: added ALS_INT, BARO_INT, ENV_I2C_SCL, ENV_I2C_SDA, VOUT1_1V8; removed none
- sheet 09_STORAGE ports: added EMMC_CLK, EMMC_CMD, EMMC_DAT0, EMMC_DAT1, EMMC_DAT2, EMMC_DAT3, EMMC_DAT4, EMMC_DAT5, EMMC_DAT6, EMMC_DAT7, EMMC_RST_N, VOUT1_1V8, VOUT2_3V0_PROVISIONAL; removed none
- sheet 10_HAPTICS ports: added HAPTIC_I2C_SCL, HAPTIC_I2C_SDA, HAPTIC_NRST, HAPTIC_TRIG_INTZ, VOUT1_1V8, VSYS; removed none
- sheet 11_BUTTONS ports: added BTN_BACK_N, BTN_DOWN_N, BTN_LIGHT_N, BTN_START_N, BTN_UP_N, VOUT1_1V8; removed none
- sheet 13_DEBUG ports: added APOLLO_RST_N, APOLLO_SWCLK, APOLLO_SWDIO, APOLLO_SWO_GPIO28, SYS_3V3, VBAT, VOUT1_1V8, VOUT2_3V0_PROVISIONAL, VSYS; removed none
- sheet 14_RF ports: added APOLLO_BLE_ANT, APOLLO_BLE_AVDD_PA, GNSS_RF, WIFI_RF; removed none

Commit message: froze schematics
Other:
- sheet 04_PPG ports: added VBAT; removed none
Changed lines of the file:
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@@
+			)
+		)
+		(pin "VBAT" passive
+			(at 345.44 86.36 0)
+			(effects
+				(font
+					(size 1.27 1.27)
+				)
 			)
 		)
@@
 		(effects
 			(font
+				(size 1.27 1.27)
+			)
+			(justify left bottom)
+		)
+	)
+	(wire
+		(pts
+			(xy 345.44 86.36) (xy 350.52 86.36)
+		)
+		(stroke
+			(width 0)
+			(type default)
+		)
+	)
+	(label "VBAT"
+		(at 350.52 86.36 0)
+		(effects
+			(font
