File: 01_APOLLO510B.kicad_sch (KiCad schematic)
At the start: 48 parts, among them U101 AP510BFA-CBR, U102 SN74AXC8T245, U103 TXB0101DRLR, U104 SN74AXC1T45, U105 SN74AXC1T45, U106 PCA9306DCU, Y101 ABS06-32.768KHZ-6-1-T, Y102 NX1612SA-48M-EXS00A-CS14265

Commit message: fix(pcb): foundation correction round 5 closure
Parts:
- Y101: footprint Crystal:Crystal_SMD_2012-2Pin_2.0x1.2mm -> sportwatch_custom:Crystal_SMD_ABS06_2.0x1.2mm
Changed lines of the file:
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@@
 			)
 		)
-		(property "Footprint" "Crystal:Crystal_SMD_2012-2Pin_2.0x1.2mm"
+		(property "Footprint" "sportwatch_custom:Crystal_SMD_ABS06_2.0x1.2mm"
 			(at 340 104 0)
 			(hide yes)

Commit message: foundation correction
Parts:
- C101, C102, C103, C104, C105, C106, C107, C108, C109, C110, C111, C112, C113, C114, C115, C116, C117, C118, C119, C120, C121, C122, C123, C124, C125, C126, C127, C128, L101, R101, R102, R103, R104, R105, R106, R107, R108, R109, R110, R111, U101, U102, U103, U104, U105, U106, Y101, Y102: Board (none) -> MAIN
