File: 03_DISPLAY.kicad_sch (KiCad schematic)
At the start: 0 parts

Commit message: updated schematics
Parts:
- added J1: ZC-A1D43W-046, sportwatch_custom:OK-23GF024-04, symbol sportwatch_display:ZC-A1D43W-046
- added R301, R302: 3.6k, Resistor_SMD:R_0402_1005Metric, symbol Device:R
- added R303, R304: 100k, Resistor_SMD:R_0402_1005Metric, symbol Device:R
- added R305, R306: 10k, Resistor_SMD:R_0402_1005Metric, symbol Device:R
Connections:
- new net DISP_QSPI_CLK: J1.5 (SPI_CLK)
- new net DISP_QSPI_CS: J1.4 (SPI_CS), R305.2
- new net DISP_QSPI_IO0: J1.7 (SPI_SI00)
- new net DISP_QSPI_IO1: J1.6 (SPI_I01)
- new net DISP_QSPI_IO2: J1.23 (SPI_SI02)
- new net DISP_QSPI_IO3: J1.22 (SPI_SI03)
- new net DISP_RST: J1.1 (LCD_RST), R303.1
- new net DISP_TE: J1.3 (TE)
- new net DISP_VCI_EN: J1.24 (VCI_EN), R306.1
- new net GND: J1.13 (GND), J1.14 (GND), J1.2 (GND), J1.21 (GND), J1.8 (GND), R303.2, R304.2, R306.2
- new net SYS_3V3: J1.15 (VDD), J1.16 (TP_VDD), R301.1, R302.1, R305.1
- new net TOUCH_INT: J1.17 (TP_INT)
- new net TOUCH_RST: J1.18 (TP_RST), R304.1
- new net TOUCH_SCL: J1.20 (TP_SCL), R302.2
- new net TOUCH_SDA: J1.19 (TP_SDA), R301.2
- new net VSYS: J1.11 (VBAT), J1.12 (VBAT)
- no-connect marks 0 -> 2
Other:
- title: (none) -> Rev-A — ZC-A1D43W-046 AMOLED / touch

Commit message: foundation correction
Parts:
- J1, R301, R302, R303, R304, R305, R306: Board (none) -> MAIN
Changed lines of the file:
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@@
 			)
 		)
-	)
+(property "Board" "MAIN" (at 0 0 0) (effects (font (size 1 1)) (hide yes)))
+)
 	(symbol
 		(lib_id "sportwatch_display:ZC-A1D43W-046")
@@
 			)
 		)
-	)
+(property "Board" "MAIN" (at 0 0 0) (effects (font (size 1 1)) (hide yes)))
+)
 	(symbol
 		(lib_id "power:GND")
@@
 			)
 		)
-	)
+(property "Board" "MAIN" (at 0 0 0) (effects (font (size 1 1)) (hide yes)))
+)
 	(symbol
 		(lib_id "power:GND")
@@
 			)
 		)
-	)
+(property "Board" "MAIN" (at 0 0 0) (effects (font (size 1 1)) (hide yes)))
+)
 	(symbol
 		(lib_id "power:GND")
@@
 			)
 		)
-	)
+(property "Board" "MAIN" (at 0 0 0) (effects (font (size 1 1)) (hide yes)))
+)
 	(symbol
 		(lib_id "Device:R")
@@
 			)
 		)
-	)
+(property "Board" "MAIN" (at 0 0 0) (effects (font (size 1 1)) (hide yes)))
+)
 	(symbol
 		(lib_id "Device:R")
@@
 			)
 		)
-	)
+(property "Board" "MAIN" (at 0 0 0) (effects (font (size 1 1)) (hide yes)))
+)
 	(symbol
 		(lib_id "Device:R")
@@
 			)
 		)
-	)
+(property "Board" "MAIN" (at 0 0 0) (effects (font (size 1 1)) (hide yes)))
+)
 	(symbol
 		(lib_id "power:GND")
@@
 			)
 		)
-	)
+(property "Board" "MAIN" (at 0 0 0) (effects (font (size 1 1)) (hide yes)))
+)
 	(symbol
 		(lib_id "Device:R")
@@
 			)
 		)
-	)
+(property "Board" "MAIN" (at 0 0 0) (effects (font (size 1 1)) (hide yes)))
+)
 	(symbol
 		(lib_id "Device:R")
@@
 			)
 		)
-	)
-)
+(property "Board" "MAIN" (at 0 0 0) (effects (font (size 1 1)) (hide yes)))
+)
+)
