File: 04_PPG.kicad_sch (KiCad schematic)
At the start: 48 parts, among them U12 MAX86141ENP+T, U13 MAX86141ENP+T, U401 TPS631000DRLR, U402 TS5A12301E, U403 TS5A12301E, U404 TS5A12301E, U405 TS5A12301E, U406 TS5A12301E, U407 TS5A12301E

Commit message: foundation correction
Parts:
- removed C403, C404, C405, C406, C407, C408, C4102, C4202: 100nF, Capacitor_SMD:C_0402_1005Metric, symbol Device:C
- removed C4101, C4201: 22uF, Capacitor_SMD:C_0402_1005Metric, symbol Device:C
- removed C4103, C4203: 1.0uF, Capacitor_SMD:C_0402_1005Metric, symbol Device:C
- removed C4104, C4204: 10uF, Capacitor_SMD:C_0402_1005Metric, symbol Device:C
- removed D401, D402, D403, D404: SFH7018A Q65113A6157, sportwatch_custom:OSRAM_SFH7018A_2.4x2.4mm, symbol sportwatch_custom:SFH7018A
- removed D405, D406, D407: SFH4053B Q65115A1586, sportwatch_custom:OSRAM_SFH4053B_1.0x0.5mm, symbol sportwatch_custom:SFH4053B
- removed D413, D414, D423, D424: SFH2703H Q65115A2199, sportwatch_custom:OSRAM_SFH2703_3.2x2.0mm, symbol sportwatch_custom:SFH2703H
- removed NT401: PPG1_PD_GND_TIE, NetTie:NetTie-2_SMD_Pad0.5mm, symbol sportwatch_custom:NetTie_2
- removed NT402: PPG2_PD_GND_TIE, NetTie:NetTie-2_SMD_Pad0.5mm, symbol sportwatch_custom:NetTie_2
- removed R401, R402, R405: 100k, Resistor_SMD:R_0402_1005Metric, symbol Device:R
- removed R403, R404: 47k, Resistor_SMD:R_0402_1005Metric, symbol Device:R
- removed R408, R409: 10k, Resistor_SMD:R_0402_1005Metric, symbol Device:R
- removed U12, U13: MAX86141ENP+T, sportwatch_custom:21-100134_N201A2-1_MXM, symbol 2026-09-16_07-42-39:MAX86141ENP+T
- removed U402, U403, U404, U405, U406, U407: TS5A12301E, Package_BGA:Texas_DSBGA-6_0.76x1.16mm_Layout2x3_P0.4mm, symbol sportwatch_custom:TS5A12301E
- added J1501: SENSOR_24_ABSTRACT, symbol Connector_Generic:Conn_01x24
- C401, C402, L401, R406, R407, U401: Board (none) -> MAIN
Connections:
- net GND: now also J1501.1 (Pin_1), J1501.10 (Pin_10), J1501.14 (Pin_14), J1501.17 (Pin_17), J1501.19 (Pin_19), J1501.20 (Pin_20), J1501.24 (Pin_24), J1501.3 (Pin_3), J1501.5 (Pin_5), J1501.7 (Pin_7)
- net PPG1_CS_N: now also J1501.8 (Pin_8)
- net PPG1_INT_N: now also J1501.11 (Pin_11)
- net PPG2_CS_N: now also J1501.9 (Pin_9)
- net PPG2_INT_N: now also J1501.12 (Pin_12)
- net PPG_SAMPLE_SYNC: now also J1501.13 (Pin_13)
- net PPG_SPI_MISO: now also J1501.6 (Pin_6)
- net PPG_SPI_MOSI: now also J1501.4 (Pin_4)
- net PPG_SPI_SCLK: now also J1501.2 (Pin_2)
- net PPG_VLED: now also J1501.21 (Pin_21), J1501.22 (Pin_22), J1501.23 (Pin_23)
- net VOUT1_1V8: now also J1501.18 (Pin_18)
- net Net-(U401-LX2): now reaches L401.2, U401.2 (LX2)
- net Net-(U401-LX1): now reaches L401.1, U401.3 (LX1)
- new net ENV_I2C_SCL: J1501.15 (Pin_15)
- new net ENV_I2C_SDA: J1501.16 (Pin_16)
- no-connect marks 3 -> 0
Other:
- note added: "Board ownership and interfaces: design/interfaces/main_rear_interface.md"
- note added: "Converter feedback and C402 stay on MAIN. Rear bypass and entry reservoir are separate."
- note added: "Optional source damping: reserve MAIN SCLK/MOSI/CS1/CS2 and REAR MISO sites; bypass in Phase 1. Values/fit require waveform ECO."
- note added: "Positions are abstract contract IDs. No connector MPN/footprint/mating permutation selected."
- note removed: "04_PPG — DUAL MAX86141 OPTICAL HR / SpO2 FRONT END — REV A"
- note removed: "AFE architecture: both MAX86141 devices share SPI SCLK/MOSI/MISO; each has its own CS and active-low open-drain INT."
- note removed: "APPLE-INSPIRED 12-EMITTER PPG: 4x green, 4x red, 3x IR850, 1x IR940. Current Apple Ultra 4 exact emitter count is not publicly enumerated; this follows the documented Ultra/Ultra 2 wavelength mix within dual-MAX86141 12-LED capability."
- note removed: "Apple-inspired optical architecture: 12 independently selected emitters total = 4 green + 4 red + 3 IR850 + 1 IR940, with the existing four SFH2703H photodiodes. Each MAX86141 uses a 3x2:1 LED mux bank."
- note removed: "C401 22uF input, C402 47uF output + existing 10uF per AFE; R406 604k/R407 91k; L401 1uH DFE252012P-1R0M=P2 baseline."
- note removed: "CRITICAL PCB: fully shield each PD_IN with its corresponding PD_GND; no unrelated traces/vias through or over the PD_GND shield. Keep PD paths extremely short."
- note removed: "Custom SFH7018A, SFH4053B, SFH2703H and TS5A12301E symbols are embedded; exact new optical/mux footprints remain for the dedicated footprint audit."
- note removed: "Firmware starting current caps: SFH4053B IR850 <=62mA; SFH7018A red <=31mA baseline; green/IR940 <=62mA baseline until optical/thermal/eye-safety validation."
- note removed: "GPIO1 of both AFEs remains PPG_SAMPLE_SYNC. Use GPIO_CTRL=1010: falling GPIO1 starts one sample; GPIO2 is automatic external-mux control (HIGH for LED1/2/3, LOW for LED4/5/6)."
- note removed: "Keep the complete PPG analog/optical region away from Wi-Fi/GNSS RF, display/high-speed buses, switchers, inductors and the haptic actuator. Optical barriers and source-detector spacing are mechanical-design items."
- note removed: "MAX86141 imported WLP footprint is retained for now. ALL three custom optical footprints plus WLP ball orientation are verified during the dedicated pre-PCB footprint audit."
- note removed: "PD_GND1/2 are separate shield/reference nets and join PCB GND only through NT401/NT402. Use real net-tie copper/footprints, not resistors, during PCB footprint/layout audit."
- note removed: "PPG VLED POWER — TPS631000 buck-boost from protected VBAT, nominal 3.82V; EN=VOUT1_1V8, MODE=GND (PFM)."
- note removed: "PPG_VLED is generated locally by U401 TPS631000 from protected VBAT. Nominal rail ~3.82 V; EN follows VOUT1_1V8. Keep VLED switching/layout away from PD_IN/PD_GND and optical analog nodes."
- note removed: "SFH7018A exact pad map embedded from OSRAM: 1/7/8 green cathode, 2/4 red+IR anode, 3 IR cathode, 5 red cathode, 6 green anode. SFH2703H symbol uses pin1 cathode, pin2 anode."
- note removed: "TS5A12301E mux logic: GPIO2 HIGH -> NO = LED1/2/3; GPIO2 LOW -> NC = LED4/5/6. Power muxes from PPG_VLED; 1.8V GPIO control is supported."
- note removed: "VDD_ANA and VDD_DIG use the same VOUT1_1V8 rail and must be shorted locally at each WLP. ADI layout guidance calls for 22uF + 0.1uF combined decoupling and 1uF on VREF."
- title: Rev-A — Optical PPG / HR / SpO2 -> MAIN - TPS631000 VLED source and rear interface
