File: 06_WIFI.kicad_sch (KiCad schematic)
At the start: 26 parts, among them U10 2.4/5GHz_DIPLEXER_TBD, U11 TPS22918DBVT, U9 NRF7002-QFAA-R7, Y1 40MHz_CL8pF_ESR100R_1612

Commit message: fix(pcb): Round 3 foundation correction — 0 DRC errors, stacked microvias, PPG ECO & guards
- Eliminate 24 committed DRC errors by refilling all zones and committing refilled state
- Rebuild 12 L1->L3 skip microvias as 24 stackup-compliant stacked L1->L2 + L2->L3 microvias (VIPPO IPC-4761 Type VII)
- Harmonize HighSpeed_50R track width to 0.100 mm across .kicad_pro, .kicad_dru, and live copper
- Execute controlled schematic ECO swapping D413 and D424 detector channels, eliminating Jordan curve crossing
- Route all 4 PPG detector channels pad-to-pad on B.Cu with continuous dedicated PD_GND ground guards
- Close schematic residuals: Y101 MPN ABS07-32.768KHZ-6-T and 8.2pF load caps, cite primary sources for Y102 and Y1 on-chip trim, cite u-blox manual for U8 VCC_RF NC
- Formally defer staged passives (eMMC interface, PPG VLED, C206) with documented reserved placement corridors
- Document comprehensive Round 3 report and update Apollo/eMMC escape matrices and AGENT_HANDOFF.md
Parts:
- Y1: value 40MHz_CL8pF_ESR100R_1612 -> NX1612SA-40M-EXS00A-CS14264
Changed lines of the file:
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@@
 			)
 		)
-		(property "Value" "40MHz_CL8pF_ESR100R_1612"
+		(property "Value" "NX1612SA-40M-EXS00A-CS14264"
 			(at 176 162.7 0)
 			(show_name no)

Commit message: foundation correction
Parts:
- C601, C602, C603, C604, C605, C606, C607, C608, C609, C610, C611, C612, C613, C614, C615, C616, C617, C618, C619, L601, R601, R602, U10, U11, U9, Y1: Board (none) -> MAIN
Changed lines of the file:
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@@
 			)
 		)
-	)
+(property "Board" "MAIN" (at 0 0 0) (effects (font (size 1 1)) (hide yes)))
+)
 	(symbol
 		(lib_id "power:GND")
@@
 			)
 		)
-	)
+(property "Board" "MAIN" (at 0 0 0) (effects (font (size 1 1)) (hide yes)))
+)
 	(symbol
 		(lib_id "Device:C")
@@
 			)
 		)
-	)
+(property "Board" "MAIN" (at 0 0 0) (effects (font (size 1 1)) (hide yes)))
+)
 	(symbol
 		(lib_id "power:GND")
@@
 			)
 		)
-	)
+(property "Board" "MAIN" (at 0 0 0) (effects (font (size 1 1)) (hide yes)))
+)
 	(symbol
 		(lib_id "Device:C")
@@
 			)
 		)
-	)
+(property "Board" "MAIN" (at 0 0 0) (effects (font (size 1 1)) (hide yes)))
+)
 	(symbol
 		(lib_id "Device:C")
@@
 			)
 		)
-	)
+(property "Board" "MAIN" (at 0 0 0) (effects (font (size 1 1)) (hide yes)))
+)
 	(symbol
 		(lib_id "power:GND")
@@
 			)
 		)
-	)
+(property "Board" "MAIN" (at 0 0 0) (effects (font (size 1 1)) (hide yes)))
+)
 	(symbol
 		(lib_id "power:GND")
@@
 			)
 		)
-	)
+(property "Board" "MAIN" (at 0 0 0) (effects (font (size 1 1)) (hide yes)))
+)
 	(symbol
 		(lib_id "power:GND")
@@
 			)
 		)
-	)
+(property "Board" "MAIN" (at 0 0 0) (effects (font (size 1 1)) (hide yes)))
+)
 	(symbol
 		(lib_id "Device:C")
@@
 			)
 		)
-	)
+(property "Board" "MAIN" (at 0 0 0) (effects (font (size 1 1)) (hide yes)))
+)
 	(symbol
 		(lib_id "Device:C")
@@
 			)
 		)
-	)
+(property "Board" "MAIN" (at 0 0 0) (effects (font (size 1 1)) (hide yes)))
+)
 	(symbol
 		(lib_id "Device:C")
@@
 			)
 		)
-	)
+(property "Board" "MAIN" (at 0 0 0) (effects (font (size 1 1)) (hide yes)))
+)
 	(symbol
 		(lib_id "sportwatch_custom:INDUCTOR_2PIN")
@@
 			)
 		)
-	)
+(property "Board" "MAIN" (at 0 0 0) (effects (font (size 1 1)) (hide yes)))
+)
 	(symbol
 		(lib_id "power:GND")
@@
 			)
 		)
-	)
+(property "Board" "MAIN" (at 0 0 0) (effects (font (size 1 1)) (hide yes)))
+)
 	(symbol
 		(lib_id "Device:C")
@@
 			)
 		)
-	)
+(property "Board" "MAIN" (at 0 0 0) (effects (font (size 1 1)) (hide yes)))
+)
 	(symbol
 		(lib_id "power:GND")
@@
 			)
 		)
-	)
+(property "Board" "MAIN" (at 0 0 0) (effects (font (size 1 1)) (hide yes)))
+)
 	(symbol
 		(lib_id "Device:C")
@@
 			)
 		)
-	)
+(property "Board" "MAIN" (at 0 0 0) (effects (font (size 1 1)) (hide yes)))
+)
 	(symbol
 		(lib_id "power:GND")
@@
 			)
 		)
-	)
+(property "Board" "MAIN" (at 0 0 0) (effects (font (size 1 1)) (hide yes)))
+)
 	(symbol
 		(lib_id "Device:C")
@@
 			)
 		)
-	)
+(property "Board" "MAIN" (at 0 0 0) (effects (font (size 1 1)) (hide yes)))
+)
 	(symbol
 		(lib_id "power:GND")
@@
 			)
 		)
-	)
+(property "Board" "MAIN" (at 0 0 0) (effects (font (size 1 1)) (hide yes)))
+)
 	(symbol
 		(lib_id "Device:C")
@@
 			)
 		)
-	)
+(property "Board" "MAIN" (at 0 0 0) (effects (font (size 1 1)) (hide yes)))
+)
 	(symbol
 		(lib_id "Device:C")
@@
 			)
 		)
-	)
+(property "Board" "MAIN" (at 0 0 0) (effects (font (size 1 1)) (hide yes)))
+)
 	(symbol
 		(lib_id "power:GND")
@@
 			)
 		)
-	)
+(property "Board" "MAIN" (at 0 0 0) (effects (font (size 1 1)) (hide yes)))
+)
 	(symbol
 		(lib_id "sportwatch_custom:TPS22918DBV")
@@
 			)
 		)
-	)
+(property "Board" "MAIN" (at 0 0 0) (effects (font (size 1 1)) (hide yes)))
+)
 	(symbol
 		(lib_id "Device:C")
@@
 			)
 		)
-	)
+(property "Board" "MAIN" (at 0 0 0) (effects (font (size 1 1)) (hide yes)))
+)
 	(symbol
 		(lib_id "power:GND")
@@
 			)
 		)
-	)
+(property "Board" "MAIN" (at 0 0 0) (effects (font (size 1 1)) (hide yes)))
+)
 	(symbol
 		(lib_id "power:GND")
@@
 			)
 		)
-	)
+(property "Board" "MAIN" (at 0 0 0) (effects (font (size 1 1)) (hide yes)))
+)
 	(symbol
 		(lib_id "power:GND")
@@
 			)
 		)
-	)
+(property "Board" "MAIN" (at 0 0 0) (effects (font (size 1 1)) (hide yes)))
+)
 	(symbol
 		(lib_id "sportwatch_custom:WIFI_DIPLEXER")
@@
 			)
 		)
-	)
+(property "Board" "MAIN" (at 0 0 0) (effects (font (size 1 1)) (hide yes)))
+)
 	(symbol
 		(lib_id "Device:R")
@@
 			)
 		)
-	)
+(property "Board" "MAIN" (at 0 0 0) (effects (font (size 1 1)) (hide yes)))
+)
 	(symbol
 		(lib_id "power:GND")
@@
 			)
 		)
-	)
+(property "Board" "MAIN" (at 0 0 0) (effects (font (size 1 1)) (hide yes)))
+)
 	(symbol
 		(lib_id "power:GND")
@@
 			)
 		)
-	)
+(property "Board" "MAIN" (at 0 0 0) (effects (font (size 1 1)) (hide yes)))
+)
 	(symbol
 		(lib_id "power:GND")
@@
 			)
 		)
-	)
+(property "Board" "MAIN" (at 0 0 0) (effects (font (size 1 1)) (hide yes)))
+)
 	(symbol
 		(lib_id "Device:R")
@@
 			)
 		)
-	)
+(property "Board" "MAIN" (at 0 0 0) (effects (font (size 1 1)) (hide yes)))
+)
 	(symbol
 		(lib_id "Device:C")
@@
 			)
 		)
-	)
+(property "Board" "MAIN" (at 0 0 0) (effects (font (size 1 1)) (hide yes)))
+)
 	(symbol
 		(lib_id "power:GND")
@@
 			)
 		)
-	)
+(property "Board" "MAIN" (at 0 0 0) (effects (font (size 1 1)) (hide yes)))
+)
 	(symbol
 		(lib_id "sportwatch_custom:Crystal_1612-4Pin_GND")
@@
 			)
 		)
-	)
+(property "Board" "MAIN" (at 0 0 0) (effects (font (size 1 1)) (hide yes)))
+)
 	(symbol
 		(lib_id "power:GND")
@@
 			)
 		)
-	)
+(property "Board" "MAIN" (at 0 0 0) (effects (font (size 1 1)) (hide yes)))
+)
 	(symbol
 		(lib_id "power:GND")
@@
 			)
 		)
-	)
+(property "Board" "MAIN" (at 0 0 0) (effects (font (size 1 1)) (hide yes)))
+)
 	(symbol
 		(lib_id "Device:C")
@@
 			)
 		)
-	)
+(property "Board" "MAIN" (at 0 0 0) (effects (font (size 1 1)) (hide yes)))
+)
 	(symbol
 		(lib_id "2026-09-16_06-57-34:NRF7002-QFAA-R")
@@
 			)
 		)
-	)
+(property "Board" "MAIN" (at 0 0 0) (effects (font (size 1 1)) (hide yes)))
+)
 	(symbol
 		(lib_id "power:GND")
@@
 			)
 		)
-	)
+(property "Board" "MAIN" (at 0 0 0) (effects (font (size 1 1)) (hide yes)))
+)
 	(symbol
 		(lib_id "Device:C")
@@
 			)
 		)
-	)
+(property "Board" "MAIN" (at 0 0 0) (effects (font (size 1 1)) (hide yes)))
+)
 	(symbol
 		(lib_id "Device:C")
@@
 			)
 		)
-	)
+(property "Board" "MAIN" (at 0 0 0) (effects (font (size 1 1)) (hide yes)))
+)
 	(symbol
 		(lib_id "power:GND")
@@
 			)
 		)
-	)
+(property "Board" "MAIN" (at 0 0 0) (effects (font (size 1 1)) (hide yes)))
+)
 	(symbol
 		(lib_id "power:GND")
@@
 			)
 		)
-	)
+(property "Board" "MAIN" (at 0 0 0) (effects (font (size 1 1)) (hide yes)))
+)
 	(symbol
 		(lib_id "power:GND")
@@
 			)
 		)
-	)
+(property "Board" "MAIN" (at 0 0 0) (effects (font (size 1 1)) (hide yes)))
+)
 	(symbol
 		(lib_id "power:GND")
@@
 			)
 		)
-	)
+(property "Board" "MAIN" (at 0 0 0) (effects (font (size 1 1)) (hide yes)))
+)
 	(symbol
 		(lib_id "power:GND")
@@
 			)
 		)
-	)
+(property "Board" "MAIN" (at 0 0 0) (effects (font (size 1 1)) (hide yes)))
+)
 	(symbol
 		(lib_id "power:GND")
@@
 			)
 		)
-	)
+(property "Board" "MAIN" (at 0 0 0) (effects (font (size 1 1)) (hide yes)))
+)
 	(symbol
 		(lib_id "power:GND")
@@
 			)
 		)
-	)
+(property "Board" "MAIN" (at 0 0 0) (effects (font (size 1 1)) (hide yes)))
+)
 	(symbol
 		(lib_id "power:GND")
@@
 			)
 		)
-	)
+(property "Board" "MAIN" (at 0 0 0) (effects (font (size 1 1)) (hide yes)))
+)
 	(symbol
 		(lib_id "Device:C")
@@
 			)
 		)
-	)
+(property "Board" "MAIN" (at 0 0 0) (effects (font (size 1 1)) (hide yes)))
+)
 	(symbol
 		(lib_id "power:GND")
@@
 			)
 		)
-	)
+(property "Board" "MAIN" (at 0 0 0) (effects (font (size 1 1)) (hide yes)))
+)
 	(symbol
 		(lib_id "Device:C")
@@
 			)
 		)
-	)
+(property "Board" "MAIN" (at 0 0 0) (effects (font (size 1 1)) (hide yes)))
+)
 	(symbol
 		(lib_id "power:GND")
@@
 			)
 		)
-	)
+(property "Board" "MAIN" (at 0 0 0) (effects (font (size 1 1)) (hide yes)))
+)
 	(symbol
 		(lib_id "power:PWR_FLAG")
@@
 			)
 		)
-	)
+(property "Board" "MAIN" (at 0 0 0) (effects (font (size 1 1)) (hide yes)))
+)
 	(text "U10 is still a placeholder: current symbol pins 2/5/7 are grounded. Confirm COM, 2.4G, 5G and all GND pad numbers against the selected diplexer datasheet before PCB freeze."
 		(at 18 201 0)
