File: 10_HAPTICS.kicad_sch (KiCad schematic)
At the start: 0 parts

Commit message: updated schematics
Parts:
- added C1001, C1002: 100nF, Capacitor_SMD:C_0402_1005Metric, symbol Device:C
- added LRA1: LRA_TBD, symbol sportwatch_custom:LRA_ACTUATOR
- added R1001, R1002, R1004: 2.2k, Resistor_SMD:R_0402_1005Metric, symbol Device:R
- added R1003: 220k, Resistor_SMD:R_0402_1005Metric, symbol Device:R
- added U7: DRV2625YFFR, YFF0009AHAN, symbol 2026-09-16_06-31-04:DRV2625YFFR
Connections:
- new net: LRA1.1 (OUT+), U7.A3 (OUT+)
- new net: LRA1.2 (OUT-), U7.C3 (OUT-)
- new net GND: C1001.2, C1002.2, R1003.2, U7.B3 (GND)
- new net HAPTIC_I2C_SCL: R1002.2, U7.C1 (SCL)
- new net HAPTIC_I2C_SDA: R1001.2, U7.B1 (SDA)
- new net HAPTIC_NRST: R1003.1, U7.B2 (NRST)
- new net HAPTIC_REG: C1002.1, U7.A2 (REG)
- new net HAPTIC_TRIG_INTZ: R1004.2, U7.A1 (TRIG_INTZ)
- new net VOUT1_1V8: R1001.1, R1002.1, R1004.1
- new net VSYS: C1001.1, U7.C2 (VDD)
Other:
- note added: "10_HAPTICS — DRV2625 CLOSED-LOOP HAPTIC DRIVER + LRA — REV A"
- note added: "C1001 (VDD) and C1002 (REG) are both 100nF as required by TI. Never use REG to power another circuit."
- note added: "DRV2625 VDD is powered from VSYS (2.7–5.5 V requirement). Logic/control bus is 1.8 V."
- note added: "DRV2625 footprint imported as YFF0009AHAN; verify WLCSP/DSBGA land pattern and ball orientation during the dedicated footprint audit."
- note added: "Exact LRA part and mechanical mounting are intentionally TBD; select before PCB mechanical freeze."
- note added: "I2C address: fixed 7-bit 0x5A. R1001/R1002 = 2.2k to 1.8 V; consolidate/DNP if this bus is later shared."
- note added: "LRA1 is electrically differential between OUT+ and OUT-. Do not add a flyback diode across the actuator."
- note added: "Mechanical/layout: place LRA away from BMM350 magnetometer, GNSS antenna and PPG analog front end; mechanically couple it to the case."
- note added: "NRST high threshold is 1.41 V, so Apollo 1.8 V GPIO drive is valid. R1003 keeps DRV2625 in shutdown during host reset/boot."
- note added: "TRIG/INTZ has an internal pull-down. R1004 is DNP and is only populated if firmware uses TRIG/INTZ as an interrupt output."
- note added: "VSYS and 1.8 V labels are still child-sheet-local until the root hierarchy integration pass."
- title: (none) -> Rev-A — Haptic driver

Commit message: refactor(kicad): integrate Rev-A hierarchy and libraries
Parts:
- U7: footprint YFF0009AHAN -> sportwatch_custom:YFF0009AHAN
Changed lines of the file:
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@@
 		)
 	)
-	(label "VOUT1_1V8"
+	(hierarchical_label "VOUT1_1V8"
+		(shape passive)
 		(at 78.74 43.18 0)
 		(effects
@@
 		)
 	)
-	(label "VSYS"
+	(hierarchical_label "VSYS"
+		(shape passive)
 		(at 92.71 70.5 0)
 		(effects
@@
 		)
 	)
-	(label "HAPTIC_I2C_SCL"
+	(hierarchical_label "HAPTIC_I2C_SCL"
+		(shape bidirectional)
 		(at 92.71 95.25 180)
 		(effects
@@
 		)
 	)
-	(label "HAPTIC_NRST"
+	(hierarchical_label "HAPTIC_NRST"
+		(shape input)
 		(at 78.74 102.87 0)
 		(effects
@@
 		)
 	)
-	(label "HAPTIC_TRIG_INTZ"
+	(hierarchical_label "HAPTIC_TRIG_INTZ"
+		(shape bidirectional)
 		(at 170.18 97.79 0)
 		(effects
@@
 		)
 	)
-	(label "HAPTIC_I2C_SDA"
+	(hierarchical_label "HAPTIC_I2C_SDA"
+		(shape bidirectional)
 		(at 68.58 59.69 0)
 		(effects
@@
 			)
 		)
-		(property "Footprint" "YFF0009AHAN"
+		(property "Footprint" "sportwatch_custom:YFF0009AHAN"
 			(at 130.81 97.79 0)
 			(hide yes)

Commit message: foundation correction
Parts:
- C1001, C1002, LRA1, R1001, R1002, R1003, R1004, U7: Board (none) -> MAIN
Changed lines of the file:
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@@
 			)
 		)
-	)
+(property "Board" "MAIN" (at 0 0 0) (effects (font (size 1 1)) (hide yes)))
+)
 	(symbol
 		(lib_id "power:GND")
@@
 			)
 		)
-	)
+(property "Board" "MAIN" (at 0 0 0) (effects (font (size 1 1)) (hide yes)))
+)
 	(symbol
 		(lib_id "power:GND")
@@
 			)
 		)
-	)
+(property "Board" "MAIN" (at 0 0 0) (effects (font (size 1 1)) (hide yes)))
+)
 	(symbol
 		(lib_id "Device:R")
@@
 			)
 		)
-	)
+(property "Board" "MAIN" (at 0 0 0) (effects (font (size 1 1)) (hide yes)))
+)
 	(symbol
 		(lib_id "sportwatch_custom:LRA_ACTUATOR")
@@
 			)
 		)
-	)
+(property "Board" "MAIN" (at 0 0 0) (effects (font (size 1 1)) (hide yes)))
+)
 	(symbol
 		(lib_id "2026-09-16_06-31-04:DRV2625YFFR")
@@
 			)
 		)
-	)
+(property "Board" "MAIN" (at 0 0 0) (effects (font (size 1 1)) (hide yes)))
+)
 	(symbol
 		(lib_id "Device:R")
@@
 			)
 		)
-	)
+(property "Board" "MAIN" (at 0 0 0) (effects (font (size 1 1)) (hide yes)))
+)
 	(symbol
 		(lib_id "power:GND")
@@
 			)
 		)
-	)
+(property "Board" "MAIN" (at 0 0 0) (effects (font (size 1 1)) (hide yes)))
+)
 	(symbol
 		(lib_id "Device:C")
@@
 			)
 		)
-	)
+(property "Board" "MAIN" (at 0 0 0) (effects (font (size 1 1)) (hide yes)))
+)
 	(symbol
 		(lib_id "Device:C")
@@
 			)
 		)
-	)
+(property "Board" "MAIN" (at 0 0 0) (effects (font (size 1 1)) (hide yes)))
+)
 	(symbol
 		(lib_id "power:GND")
@@
 			)
 		)
-	)
+(property "Board" "MAIN" (at 0 0 0) (effects (font (size 1 1)) (hide yes)))
+)
 	(symbol
 		(lib_id "Device:R")
@@
 			)
 		)
-	)
-)
+(property "Board" "MAIN" (at 0 0 0) (effects (font (size 1 1)) (hide yes)))
+)
+)
