File: 12_CHARGING.kicad_sch (KiCad schematic)
At the start: 0 parts

Commit message: foundation correction
Parts:
- added D1201: ESD_TVS_RATING_MPN_TBD, symbol Device:D_TVS
- added J202: CHARGER_HARNESS_TBD, symbol Connector_Generic:Conn_01x02
- added U1201: MANDATORY_OV_REV_ILIM_MPN_TBD, symbol sportwatch_interfaces:ChargerProtection_Provision
Connections:
- new net CHG_RAW_5V: J202.1 (Pin_1), U1201.1 (RAW_IN)
- new net GND: D1201.2 (A2), J202.2 (Pin_2), U1201.3 (GND)
- new net VBUSIN: D1201.1 (A1), U1201.2 (PROTECTED_OUT)
Other:
- note added: "C201 remains on MAIN at U201 VBUS input. Charger current must not use sensor FPC, PD_GND, NT401/NT402 or optical guard copper."
- note added: "TVS alone does not solve sustained OV/reverse polarity. Provide local contact ESD diversion in dedicated CHARGER harness."
- note added: "U1201 mandatory functional protection provision. No bypass. Final implementation/MPN/ratings require dock fault envelope."
- note added: "nPM1300 PS v1.3: VBUS operational 4.0-5.5V; absolute -0.3..22V. Built-in OV isolation does not qualify negative input."
Changed lines of the file:
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@@
 	(generator_version "10.0")
 	(paper "A4")
+	(symbol (lib_id "Connector_Generic:Conn_01x02") (at 45.72 55.88 0) (unit 1) (pin "1") (pin "2") (property "Reference" "J202" (at 45.72 53.34 0) (effects (font (size 1.27 1.27)))) (instances (project "sportwatch_revA" (path "/063f9d99-6c07-44cf-ba32-e33897e06972/13f98b5d-2735-4ce5-b6a9-56134247b933" (reference "J202") (unit 1))))
+	(property "Value" "CHARGER_HARNESS_TBD" (at 45.72 60.96 0) (effects (font (size 1.27 1.27))))
+	(property "Footprint" "" (at 45.72 55.88 0) (effects (font (size 1.27 1.27)) (hide yes)))
+	(property "Board" "MAIN" (at 45.72 55.88 0) (effects (font (size 1.27 1.27)) (hide yes)))
+	(property "SelectionStatus" "PROVISIONAL - MPN and footprint TBD" (at 45.72 55.88 0) (effects (font (size 1.27 1.27)) (hide yes)))
+	(property "Contract" "pin1=CHG_RAW_5V; pin2=GND; external contacts separate" (at 45.72 55.88 0) (effects (font (size 1.27 1.27)) (hide yes))))
+	(global_label "CHG_RAW_5V" (shape input) (at 40.64 55.88 180) (effects (font (size 1.27 1.27)) (justify right)))
+	(global_label "GND" (shape input) (at 40.64 58.42 180) (effects (font (size 1.27 1.27)) (justify right)))
+	(symbol (lib_id "sportwatch_interfaces:ChargerProtection_Provision") (at 121.92 55.88 0) (unit 1) (pin "1") (pin "2") (pin "3") (property "Reference" "U1201" (at 121.92 46.99 0) (effects (font (size 1.27 1.27)))) (instances (project "sportwatch_revA" (path "/063f9d99-6c07-44cf-ba32-e33897e06972/13f98b5d-2735-4ce5-b6a9-56134247b933" (reference "U1201") (unit 1))))
+	(property "Value" "MANDATORY_OV_REV_ILIM_MPN_TBD" (at 121.92 69.85 0) (effects (font (size 1.27 1.27))))
+	(property "Footprint" "" (at 121.92 55.88 0) (effects (font (size 1.27 1.27)) (hide yes)))
+	(property "Board" "MAIN" (at 121.92 55.88 0) (effects (font (size 1.27 1.27)) (hide yes)))
+	(property "SelectionStatus" "PROVISIONAL - MPN and footprint TBD" (at 121.92 55.88 0) (effects (font (size 1.27 1.27)) (hide yes)))
+	(property "Implementation" "Functional provision, not a selected IC; must implement OV disconnect, reverse polarity/reverse current block, current/fault limit" (at 121.92 55.88 0) (effects (font (size 1.27 1.27)) (hide yes))))
+	(global_label "CHG_RAW_5V" (shape input) (at 104.14 55.88 180) (effects (font (size 1.27 1.27)) (justify right)))
+	(global_label "VBUSIN" (shape input) (at 139.7 55.88 0) (effects (font (size 1.27 1.27)) (justify left)))
+	(global_label "GND" (shape input) (at 121.92 68.58 270) (effects (font (size 1.27 1.27)) (justify right)))
+	(symbol (lib_id "Device:D_TVS") (at 198.12 55.88 0) (unit 1) (pin "1") (pin "2") (property "Reference" "D1201" (at 198.12 53.34 0) (effects (font (size 1.27 1.27)))) (instances (project "sportwatch_revA" (path "/063f9d99-6c07-44cf-ba32-e33897e06972/13f98b5d-2735-4ce5-b6a9-56134247b933" (reference "D1201") (unit 1))))
+	(property "Value" "ESD_TVS_RATING_MPN_TBD" (at 198.12 58.42 0) (effects (font (size 1.27 1.27))))
+	(property "Footprint" "" (at 198.12 55.88 0) (effects (font (size 1.27 1.27)) (hide yes)))
+	(property "Board" "MAIN" (at 198.12 55.88 0) (effects (font (size 1.27 1.27)) (hide yes)))
+	(property "SelectionStatus" "PROVISIONAL - MPN and footprint TBD" (at 198.12 55.88 0) (effects (font (size 1.27 1.27)) (hide yes)))
+	(property "Qualification" "Recommended normal VBUS 4.0-5.5V; absolute stress limits -0.3..22V. Positive transient overshoot shall remain below 22V and negative transient/reverse protection shall keep PMIC VBUS at or above -0.3V with design margin. Sustained reverse voltage requires series blocking; final clamps and series protection remain TBD against qualified dock/fault envelope; TVS standoff above dock maximum." (at 198.12 55.88 0) (effects (font (size 1.27 1.27)) (hide yes))))
+	(global_label "VBUSIN" (shape input) (at 194.31 55.88 180) (effects (font (size 1.27 1.27)) (justify right)))
+	(global_label "GND" (shape input) (at 201.93 55.88 0) (effects (font (size 1.27 1.27)) (justify left)))
+	(symbol (lib_id "power:PWR_FLAG") (at 45.72 91.44 0) (unit 1) (pin "1") (property "Reference" "#FLG1201" (at 45.72 92.71 0) (effects (font (size 1.27 1.27)) (hide yes))) (instances (project "sportwatch_revA" (path "/063f9d99-6c07-44cf-ba32-e33897e06972/13f98b5d-2735-4ce5-b6a9-56134247b933" (reference "#FLG1201") (unit 1))))
+	(property "Value" "PWR_FLAG" (at 45.72 87.63 0) (effects (font (size 1.27 1.27))))
+	(property "Footprint" "" (at 45.72 91.44 0) (effects (font (size 1.27 1.27)) (hide yes)))
+	(property "Board" "MAIN" (at 45.72 91.44 0) (effects (font (size 1.27 1.27)) (hide yes)))
+	(property "SelectionStatus" "PROVISIONAL - MPN and footprint TBD" (at 45.72 91.44 0) (effects (font (size 1.27 1.27)) (hide yes)))
+	(property "Source" "External current-limited +5V dock via separate harness" (at 45.72 91.44 0) (effects (font (size 1.27 1.27)) (hide yes))))
+	(global_label "CHG_RAW_5V" (shape input) (at 45.72 91.44 270) (effects (font (size 1.27 1.27)) (justify right)))
+	(text "U1201 mandatory functional protection provision. No bypass. Final implementation/MPN/ratings require dock fault envelope." (at 12.7 127 0) (effects (justify left bottom) (font (size 0.9 0.9))))
+	(text "nPM1300 PS v1.3: VBUS operational 4.0-5.5V; absolute -0.3..22V. Built-in OV isolation does not qualify negative input." (at 12.7 139.7 0) (effects (justify left bottom) (font (size 0.9 0.9))))
+	(text "TVS alone does not solve sustained OV/reverse polarity. Provide local contact ESD diversion in dedicated CHARGER harness." (at 12.7 152.4 0) (effects (justify left bottom) (font (size 0.9 0.9))))
+	(text "C201 remains on MAIN at U201 VBUS input. Charger current must not use sensor FPC, PD_GND, NT401/NT402 or optical guard copper." (at 12.7 165.1 0) (effects (justify left bottom) (font (size 0.9 0.9))))
 )
