File: 14_RF.kicad_sch (KiCad schematic)
At the start: 0 parts

Commit message: fixed schematics errors
Parts:
- added AE1401: ANT_BLE_2G4_TBD, symbol sportwatch_custom:ANTENNA_TBD
- added AE1410: ANT_WIFI_2G4_5G_TBD, symbol sportwatch_custom:ANTENNA_TBD
- added AE1420: ANT_GNSS_L1_L5_TBD, symbol sportwatch_custom:ANTENNA_TBD
- added C1401: 18pF, Capacitor_SMD:C_0201_0603Metric, symbol Device:C
- added C1402: 2.8pF, Capacitor_SMD:C_0201_0603Metric, symbol Device:C
- added C1403: 3.2pF, Capacitor_SMD:C_0201_0603Metric, symbol Device:C
- added C1404: 1.0pF DNP, Capacitor_SMD:C_0201_0603Metric, symbol Device:C
- added C1405: 220pF, Capacitor_SMD:C_0201_0603Metric, symbol Device:C
- added C1410, C1411, C1420, C1421: DNP, Capacitor_SMD:C_0201_0603Metric, symbol Device:C
- added L1401: 1.5nH, symbol sportwatch_custom:RF_INDUCTOR
- added L1402: 1.8nH, symbol sportwatch_custom:RF_INDUCTOR
- added R1401: 0R (Lm2 tune), Resistor_SMD:R_0201_0603Metric, symbol Device:R
- added R1410, R1420: 0R, Resistor_SMD:R_0201_0603Metric, symbol Device:R
- added TP1401: BLE_RF_TEST_TBD, symbol sportwatch_custom:RF_TEST_PROVISION
- added TP1410: WIFI_RF_TEST_TBD, symbol sportwatch_custom:RF_TEST_PROVISION
- added TP1420: GNSS_RF_TEST_TBD, symbol sportwatch_custom:RF_TEST_PROVISION
Connections:
- new net: C1403.1, L1402.2, R1401.1
- new net: C1404.1, C1405.1, R1401.2
- new net APOLLO_BLE_ANT: C1402.1, L1401.1, L1402.1
- new net APOLLO_BLE_AVDD_PA: C1401.1, L1401.2
- new net BLE_RF_50R: AE1401.1 (RF), C1405.2, TP1401.1 (RF)
- new net GND: C1401.2, C1402.2, C1403.2, C1404.2, C1410.2, C1411.2, C1420.2, C1421.2
- new net GNSS_ANT_50R: AE1420.1 (RF), C1421.1, R1420.2, TP1420.1 (RF)
- new net GNSS_RF: C1420.1, R1420.1
- new net WIFI_ANT_50R: AE1410.1 (RF), C1411.1, R1410.2, TP1410.1 (RF)
- new net WIFI_RF: C1410.1, R1410.1
Other:
- note added: "14_RF — ANTENNA INTERFACES / MATCHING / TUNING — REV A"
- note added: "APOLLO510B BLE 2.4 GHz"
- note added: "All RF paths must be controlled 50-ohm transmission lines with continuous reference ground, short feeds, via fencing where appropriate, and no unrelated routing through antenna keepouts."
- note added: "BLE R1401 is the optional Lm2 position populated as 0R for Rev-A baseline; C1402 is on ANT/Lm1 input, C1403 at Lm1/Lm2 junction, C1404 DNP at Lm2 output."
- note added: "BLE initial values are tuning STARTING POINTS only: LDC 1.5nH, Cdc1 18pF, Lm1 2.4nH, Cm1 2.0pF, Cm2 2.0pF, Cm3 DNP, Cc1 220pF. Final values require VNA/RF tuning on the real watch geometry."
- note added: "BLE: N1 BLE_ANT is single-ended RF; M1 BLE_AVDD_PA feeds the PA bias network. L1401/C1401 and the matching chain follow Ambiq's published initial BLE topology."
- note added: "Child-sheet labels APOLLO_BLE_ANT / APOLLO_BLE_AVDD_PA / WIFI_RF / GNSS_RF must be exported through the final hierarchy integration."
- note added: "Exact BLE/Wi-Fi/GNSS antennas are selected before routing is frozen, after the board outline, display, battery, case/bezel and available perimeter/ground-clearance regions are known."
- note added: "Exact antenna MPNs/footprints are intentionally frozen only after case + PCB outline + battery + display geometry are known."
- note added: "If the final 50-mm-class mechanics cannot support three independent antennas, BLE/Wi-Fi sharing may be reconsidered, but that requires a deliberate RF switch/diplexer redesign; do not silently merge the feeds."
- note added: "Keep GNSS especially far from display clocks, Wi-Fi, switching regulators and haptic currents. Final antenna placements/keepouts are mechanical + RF decisions, not schematic-only decisions."
- note added: "MAX-F10S GNSS L1/L5 — passive dual-band antenna baseline"
- note added: "MAX-F10S RF_IN is internally DC-blocked and requires a 50-ohm feed. No extra DC-block capacitor or active-antenna bias network is fitted for the passive Rev-A baseline."
- note added: "TP1401/TP1410/TP1420 are electrically attached RF test PROVISIONS; implement as tiny low-stub probe/coax-switch structures during PCB RF layout."
- note added: "Wi-Fi and GNSS use DNP/0R/DNP pi footprints so the antenna feed can be tuned without a PCB respin. Exact capacitor/series element values are selected after antenna and enclosure freeze."
- note added: "Wi-Fi: 06_WIFI already combines nRF7002 TXRF0/TXRF1 through the Nordic 2.4/5GHz diplexer. 14_RF therefore starts from the single WIFI_RF feed."
- note added: "nRF7002 Wi-Fi 2.4 / 5 GHz — WIFI_RF is already after the Nordic diplexer on 06_WIFI"
- title: (none) -> Rev-A — RF / Antenna Networks

Commit message: refactor(kicad): integrate Rev-A hierarchy and libraries
Changed lines of the file:
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@@
 		)
 	)
-	(label "APOLLO_BLE_ANT"
+	(hierarchical_label "APOLLO_BLE_ANT"
+		(shape passive)
 		(at 30 48 180)
 		(effects
@@
 		)
 	)
-	(label "WIFI_RF"
+	(hierarchical_label "WIFI_RF"
+		(shape passive)
 		(at 30 103 180)
 		(effects
@@
 		)
 	)
-	(label "APOLLO_BLE_AVDD_PA"
+	(hierarchical_label "APOLLO_BLE_AVDD_PA"
+		(shape passive)
 		(at 62 61 0)
 		(effects
@@
 		)
 	)
-	(label "GNSS_RF"
+	(hierarchical_label "GNSS_RF"
+		(shape passive)
 		(at 30 157 180)
 		(effects

Commit message: feat(kicad): assign and audit Rev-A footprints
Parts:
- L1401, L1402: footprint (none) -> Inductor_SMD:L_0201_0603Metric
Changed lines of the file:
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@@
 			)
 		)
-		(property "Footprint" ""
+		(property "Footprint" "Inductor_SMD:L_0201_0603Metric"
 			(at 76 48 0)
 			(hide yes)
@@
 			)
 		)
-		(property "Footprint" ""
+		(property "Footprint" "Inductor_SMD:L_0201_0603Metric"
 			(at 48 61 0)
 			(hide yes)

Commit message: foundation correction
Parts:
- AE1401, AE1410, AE1420, C1401, C1402, C1403, C1404, C1405, C1410, C1411, C1420, C1421, L1401, L1402, R1401, R1410, R1420, TP1401, TP1410, TP1420: Board (none) -> MAIN
Changed lines of the file:
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@@
 			)
 		)
-	)
+(property "Board" "MAIN" (at 0 0 0) (effects (font (size 1 1)) (hide yes)))
+)
 	(symbol
 		(lib_id "sportwatch_custom:ANTENNA_TBD")
@@
 			)
 		)
-	)
+(property "Board" "MAIN" (at 0 0 0) (effects (font (size 1 1)) (hide yes)))
+)
 	(symbol
 		(lib_id "sportwatch_custom:ANTENNA_TBD")
@@
 			)
 		)
-	)
+(property "Board" "MAIN" (at 0 0 0) (effects (font (size 1 1)) (hide yes)))
+)
 	(symbol
 		(lib_id "Device:C")
@@
 			)
 		)
-	)
+(property "Board" "MAIN" (at 0 0 0) (effects (font (size 1 1)) (hide yes)))
+)
 	(symbol
 		(lib_id "sportwatch_custom:RF_TEST_PROVISION")
@@
 			)
 		)
-	)
+(property "Board" "MAIN" (at 0 0 0) (effects (font (size 1 1)) (hide yes)))
+)
 	(symbol
 		(lib_id "Device:R")
@@
 			)
 		)
-	)
+(property "Board" "MAIN" (at 0 0 0) (effects (font (size 1 1)) (hide yes)))
+)
 	(symbol
 		(lib_id "power:GND")
@@
 			)
 		)
-	)
+(property "Board" "MAIN" (at 0 0 0) (effects (font (size 1 1)) (hide yes)))
+)
 	(symbol
 		(lib_id "sportwatch_custom:RF_TEST_PROVISION")
@@
 			)
 		)
-	)
+(property "Board" "MAIN" (at 0 0 0) (effects (font (size 1 1)) (hide yes)))
+)
 	(symbol
 		(lib_id "sportwatch_custom:RF_INDUCTOR")
@@
 			)
 		)
-	)
+(property "Board" "MAIN" (at 0 0 0) (effects (font (size 1 1)) (hide yes)))
+)
 	(symbol
 		(lib_id "sportwatch_custom:RF_INDUCTOR")
@@
 			)
 		)
-	)
+(property "Board" "MAIN" (at 0 0 0) (effects (font (size 1 1)) (hide yes)))
+)
 	(symbol
 		(lib_id "power:GND")
@@
 			)
 		)
-	)
+(property "Board" "MAIN" (at 0 0 0) (effects (font (size 1 1)) (hide yes)))
+)
 	(symbol
 		(lib_id "sportwatch_custom:RF_TEST_PROVISION")
@@
 			)
 		)
-	)
+(property "Board" "MAIN" (at 0 0 0) (effects (font (size 1 1)) (hide yes)))
+)
 	(symbol
 		(lib_id "power:GND")
@@
 			)
 		)
-	)
+(property "Board" "MAIN" (at 0 0 0) (effects (font (size 1 1)) (hide yes)))
+)
 	(symbol
 		(lib_id "Device:C")
@@
 			)
 		)
-	)
+(property "Board" "MAIN" (at 0 0 0) (effects (font (size 1 1)) (hide yes)))
+)
 	(symbol
 		(lib_id "Device:C")
@@
 			)
 		)
-	)
+(property "Board" "MAIN" (at 0 0 0) (effects (font (size 1 1)) (hide yes)))
+)
 	(symbol
 		(lib_id "Device:C")
@@
 			)
 		)
-	)
+(property "Board" "MAIN" (at 0 0 0) (effects (font (size 1 1)) (hide yes)))
+)
 	(symbol
 		(lib_id "Device:C")
@@
 			)
 		)
-	)
+(property "Board" "MAIN" (at 0 0 0) (effects (font (size 1 1)) (hide yes)))
+)
 	(symbol
 		(lib_id "sportwatch_custom:ANTENNA_TBD")
@@
 			)
 		)
-	)
+(property "Board" "MAIN" (at 0 0 0) (effects (font (size 1 1)) (hide yes)))
+)
 	(symbol
 		(lib_id "Device:C")
@@
 			)
 		)
-	)
+(property "Board" "MAIN" (at 0 0 0) (effects (font (size 1 1)) (hide yes)))
+)
 	(symbol
 		(lib_id "Device:C")
@@
 			)
 		)
-	)
+(property "Board" "MAIN" (at 0 0 0) (effects (font (size 1 1)) (hide yes)))
+)
 	(symbol
 		(lib_id "power:GND")
@@
 			)
 		)
-	)
+(property "Board" "MAIN" (at 0 0 0) (effects (font (size 1 1)) (hide yes)))
+)
 	(symbol
 		(lib_id "power:GND")
@@
 			)
 		)
-	)
+(property "Board" "MAIN" (at 0 0 0) (effects (font (size 1 1)) (hide yes)))
+)
 	(symbol
 		(lib_id "power:GND")
@@
 			)
 		)
-	)
+(property "Board" "MAIN" (at 0 0 0) (effects (font (size 1 1)) (hide yes)))
+)
 	(symbol
 		(lib_id "Device:C")
@@
 			)
 		)
-	)
+(property "Board" "MAIN" (at 0 0 0) (effects (font (size 1 1)) (hide yes)))
+)
 	(symbol
 		(lib_id "power:GND")
@@
 			)
 		)
-	)
+(property "Board" "MAIN" (at 0 0 0) (effects (font (size 1 1)) (hide yes)))
+)
 	(symbol
 		(lib_id "power:GND")
@@
 			)
 		)
-	)
+(property "Board" "MAIN" (at 0 0 0) (effects (font (size 1 1)) (hide yes)))
+)
 	(symbol
 		(lib_id "Device:R")
@@
 			)
 		)
-	)
+(property "Board" "MAIN" (at 0 0 0) (effects (font (size 1 1)) (hide yes)))
+)
 	(symbol
 		(lib_id "Device:C")
@@
 			)
 		)
-	)
-)
+(property "Board" "MAIN" (at 0 0 0) (effects (font (size 1 1)) (hide yes)))
+)
+)
