File: sportwatch_revA.kicad_pcb (KiCad board)
At the start: 8 copper layers, 46 x 46 mm, 228 parts, among them J1 ZC-A1D43W-046, J1301 TC2030-CTX-NL_TARGET, U101 AP510BFA-CBR, U102 SN74AXC8T245, U103 TXB0101DRLR, U104 SN74AXC1T45, U105 SN74AXC1T45, U106 PCA9306DCU, U11 TPS22918DBVT, U12 MAX86141ENP+T, U13 MAX86141ENP+T, U201 nPM1300-QEXX, U202 TPS63900, U4 BMP585, U401 TPS631000DRLR, U402 TS5A12301E, U403 TS5A12301E, U404 TS5A12301E, U405 TS5A12301E, U406 TS5A12301E, U407 TS5A12301E, U5 OPT4001DTSR, U6 MAX30208CLB+T, U7 DRV2625YFFR, U702 LSM6DSV16XTR, U703 BMM350, U8 MAX-F10S-00B, U9 NRF7002-QFAA-R7, U901 EMMC64G-TB9F-06011, Y1 40MHz_CL8pF_ESR100R_1612, Y101 32.768kHz / low-CL TBD, Y102 48MHz / CL=8-11pF / ESR<=60R

Commit message: fix(pcb): Round 3 foundation correction — 0 DRC errors, stacked microvias, PPG ECO & guards
- Eliminate 24 committed DRC errors by refilling all zones and committing refilled state
- Rebuild 12 L1->L3 skip microvias as 24 stackup-compliant stacked L1->L2 + L2->L3 microvias (VIPPO IPC-4761 Type VII)
- Harmonize HighSpeed_50R track width to 0.100 mm across .kicad_pro, .kicad_dru, and live copper
- Execute controlled schematic ECO swapping D413 and D424 detector channels, eliminating Jordan curve crossing
- Route all 4 PPG detector channels pad-to-pad on B.Cu with continuous dedicated PD_GND ground guards
- Close schematic residuals: Y101 MPN ABS07-32.768KHZ-6-T and 8.2pF load caps, cite primary sources for Y102 and Y1 on-chip trim, cite u-blox manual for U8 VCC_RF NC
- Formally defer staged passives (eMMC interface, PPG VLED, C206) with documented reserved placement corridors
- Document comprehensive Round 3 report and update Apollo/eMMC escape matrices and AGENT_HANDOFF.md
Connections:
- D413 pad 1: /04_PPG/PPG1_PD1_IN -> /04_PPG/PPG2_PD2_IN
- D413 pad 2: /04_PPG/PPG1_PD_GND -> /04_PPG/PPG2_PD_GND
- D424 pad 1: /04_PPG/PPG2_PD2_IN -> /04_PPG/PPG1_PD1_IN
- D424 pad 2: /04_PPG/PPG2_PD_GND -> /04_PPG/PPG1_PD_GND
Routing:
- net /04_PPG/PPG1_PD_GND: track 7.83 -> 19.3 mm
- net /04_PPG/PPG2_PD_GND: track 18.1 -> 28.6 mm
- net /04_PPG/PPG2_PD2_IN: track 0.00 -> 7.50 mm
- net /04_PPG/PPG1_PD1_IN: track 0.00 -> 6.68 mm
- net /EMMC_DAT6: vias 2 -> 4
- net /EMMC_DAT5: vias 2 -> 4
- net /EMMC_DAT4: vias 2 -> 4
- net /EMMC_CMD: vias 2 -> 4
- net /EMMC_CLK: vias 2 -> 4
- net /01_APOLLO510B/MCU_EMMC_CLK: vias 2 -> 4
Changed lines of the file:
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@@
 			(layers "B.Cu" "B.Mask" "B.Paste")
 			(roundrect_rratio 0.2)
-			(net "/04_PPG/PPG1_PD1_IN")
+			(net "/04_PPG/PPG2_PD2_IN")
 			(pinfunction "CATHODE_1")
 			(pintype "passive")
@@
 			(layers "B.Cu" "B.Mask" "B.Paste")
 			(roundrect_rratio 0.2)
-			(net "/04_PPG/PPG1_PD_GND")
+			(net "/04_PPG/PPG2_PD_GND")
 			(pinfunction "ANODE_2")
 			(pintype "passive")
@@
 			(layers "B.Cu" "B.Mask" "B.Paste")
 			(roundrect_rratio 0.2)
-			(net "/04_PPG/PPG2_PD2_IN")
+			(net "/04_PPG/PPG1_PD1_IN")
 			(pinfunction "CATHODE_1")
 			(pintype "passive")
@@
 			(layers "B.Cu" "B.Mask" "B.Paste")
 			(roundrect_rratio 0.2)
-			(net "/04_PPG/PPG2_PD_GND")
+			(net "/04_PPG/PPG1_PD_GND")
 			(pinfunction "ANODE_2")
 			(pintype "passive")
@@
 		(size 0.22)
 		(drill 0.1)
-		(layers "F.Cu" "In2.Cu")
+		(layers "F.Cu" "In1.Cu")
 		(net "/01_APOLLO510B/MCU_EMMC_CLK")
 	)
@@
 		(size 0.22)
 		(drill 0.1)
-		(layers "F.Cu" "In2.Cu")
+		(layers "F.Cu" "In1.Cu")
+		(net "/01_APOLLO510B/MCU_EMMC_CLK")
+	)
+	(via micro
+		(at 100.8 98.7)
+		(size 0.22)
+		(drill 0.1)
+		(layers "In1.Cu" "In2.Cu")
+		(net "/01_APOLLO510B/MCU_EMMC_CLK")
+	)
+	(via micro
+		(at 101.18 101.475)
+		(size 0.22)
+		(drill 0.1)
+		(layers "In1.Cu" "In2.Cu")
 		(net "/01_APOLLO510B/MCU_EMMC_CLK")
 	)
@@
 		(size 0.22)
 		(drill 0.1)
-		(layers "F.Cu" "In2.Cu")
+		(layers "F.Cu" "In1.Cu")
 		(net "/EMMC_CLK")
 	)
@@
 		(size 0.22)
 		(drill 0.1)
-		(layers "F.Cu" "In2.Cu")
+		(layers "F.Cu" "In1.Cu")
+		(net "/EMMC_CLK")
+	)
+	(via micro
+		(at 99.25 109.25)
+		(size 0.22)
+		(drill 0.1)
+		(layers "In1.Cu" "In2.Cu")
+		(net "/EMMC_CLK")
+	)
+	(via micro
+		(at 101.82 101.475)
+		(size 0.22)
+		(drill 0.1)
+		(layers "In1.Cu" "In2.Cu")
 		(net "/EMMC_CLK")
 	)
@@
 		(size 0.22)
 		(drill 0.1)
-		(layers "F.Cu" "In2.Cu")
+		(layers "F.Cu" "In1.Cu")
+		(net "/EMMC_DAT6")
+	)
+	(via micro
+		(at 100 98.7)
+		(size 0.22)
+		(drill 0.1)
+		(layers "F.Cu" "In1.Cu")
+		(net "/EMMC_DAT6")
+	)
+	(via micro
+		(at 98.75 104.25)
+		(size 0.22)
+		(drill 0.1)
+		(layers "In1.Cu" "In2.Cu")
 		(net "/EMMC_DAT6")
 	)
@@
 		(size 0.22)
 		(drill 0.1)
-		(layers "F.Cu" "In2.Cu")
+		(layers "In1.Cu" "In2.Cu")
 		(net "/EMMC_DAT6")
 	)
@@
 	)
 	(via micro
+		(at 100 97.9)
+		(size 0.22)
+		(drill 0.1)
+		(layers "F.Cu" "In1.Cu")
+		(net "/EMMC_DAT4")
+	)
+	(via micro
+		(at 97.75 104.25)
+		(size 0.22)
+		(drill 0.1)
+		(layers "F.Cu" "In1.Cu")
+		(net "/EMMC_DAT4")
+	)
+	(via micro
 		(at 97.75 104.25)
 		(size 0.22)
 		(drill 0.1)
-		(layers "F.Cu" "In2.Cu")
+		(layers "In1.Cu" "In2.Cu")
 		(net "/EMMC_DAT4")
 	)
@@
 		(size 0.22)
 		(drill 0.1)
-		(layers "F.Cu" "In2.Cu")
+		(layers "In1.Cu" "In2.Cu")
 		(net "/EMMC_DAT4")
 	)
@@
 		(size 0.22)
 		(drill 0.1)
-		(layers "F.Cu" "In2.Cu")
+		(layers "F.Cu" "In1.Cu")
 		(net "/EMMC_DAT5")
 	)
@@
 		(size 0.22)
 		(drill 0.1)
-		(layers "F.Cu" "In2.Cu")
+		(layers "F.Cu" "In1.Cu")
+		(net "/EMMC_DAT5")
+	)
+	(via micro
+		(at 98.25 104.25)
+		(size 0.22)
+		(drill 0.1)
+		(layers "In1.Cu" "In2.Cu")
+		(net "/EMMC_DAT5")
+	)
+	(via micro
+		(at 100 98.3)
+		(size 0.22)
+		(drill 0.1)
+		(layers "In1.Cu" "In2.Cu")
 		(net "/EMMC_DAT5")
 	)
@@
 	)
 	(via micro
+		(at 100.4 98.7)
+		(size 0.22)
+		(drill 0.1)
+		(layers "F.Cu" "In1.Cu")
+		(net "/EMMC_CMD")
+	)
+	(via micro
+		(at 98.75 109.25)
+		(size 0.22)
+		(drill 0.1)
+		(layers "F.Cu" "In1.Cu")
+		(net "/EMMC_CMD")
+	)
+	(via micro
 		(at 98.75 109.25)
 		(size 0.22)
 		(drill 0.1)
-		(layers "F.Cu" "In2.Cu")
+		(layers "In1.Cu" "In2.Cu")
 		(net "/EMMC_CMD")
 	)
@@
 		(size 0.22)
 		(drill 0.1)
-		(layers "F.Cu" "In2.Cu")
+		(layers "In1.Cu" "In2.Cu")
 		(net "/EMMC_CMD")
 	)
@@
 	)
 	(segment
-		(start 101.4 106.6)
-		(end 100.8 106.6)
+		(start 101.2 100.75)
+		(end 101.2 105.8)
+		(width 0.1)
+		(layer "B.Cu")
+		(net "/04_PPG/PPG1_PD1_IN")
+	)
+	(segment
+		(start 101.95 100)
+		(end 101.2 100.75)
+		(width 0.1)
+		(layer "B.Cu")
+		(net "/04_PPG/PPG1_PD1_IN")
+	)
+	(segment
+		(start 101.2 105.8)
+		(end 100.8 106.2)
+		(width 0.1)
+		(layer "B.Cu")
+		(net "/04_PPG/PPG1_PD1_IN")
+	)
+	(segment
+		(start 101.8 106.6)
+		(end 101.8 108.5)
+		(width 0.1)
+		(layer "B.Cu")
+		(net "/04_PPG/PPG1_PD_GND")
+	)
+	(segment
+		(start 104.45 100.5)
+		(end 101.8 103.15)
 		(width 0.1)
 		(layer "B.Cu")
@@
 	)
 	(segment
-		(start 101.4 103.35)
-		(end 101.4 106.6)
+		(start 104.45 100)
+		(end 104.45 100.5)
 		(width 0.1)
 		(layer "B.Cu")
@@
 	)
 	(segment
-		(start 101.4 108.5)
+		(start 101.8 108.5)
 		(end 101.3 108.5)
 		(width 0.1)
@@
 	)
 	(segment
-		(start 101.4 106.6)
-		(end 101.4 108.5)
+		(start 100 100.5)
+		(end 101.2 98.7)
+		(width 0.1)
+		(layer "B.Cu")
+		(net "/04_PPG/PPG1_PD_GND")
+	)
+	(segment
+		(start 104.45 98.7)
+		(end 104.45 100)
 		(width 0.1)
 		(layer "B.Cu")
@@
 	(segment
 		(start 100 101.95)
-		(end 101.4 103.35)
+		(end 100 100.5)
 		(width 0.1)
 		(layer "B.Cu")
@@
 	)
 	(segment
-		(start 92.1 98.4)
-		(end 92.1 98.7)
+		(start 101.8 106.6)
+		(end 100.8 106.6)
+		(width 0.1)
+		(layer "B.Cu")
+		(net "/04_PPG/PPG1_PD_GND")
+	)
+	(segment
+		(start 101.2 98.7)
+		(end 104.45 98.7)
+		(width 0.1)
+		(layer "B.Cu")
+		(net "/04_PPG/PPG1_PD_GND")
+	)
+	(segment
+		(start 101.8 103.15)
+		(end 101.8 106.6)
+		(width 0.1)
+		(layer "B.Cu")
+		(net "/04_PPG/PPG1_PD_GND")
+	)
+	(segment
+		(start 100 98.05)
+		(end 99.5 98)
+		(width 0.1)
+		(layer "B.Cu")
+		(net "/04_PPG/PPG2_PD2_IN")
+	)
+	(segment
+		(start 99.5 98)
+		(end 92.5 98)
+		(width 0.1)
+		(layer "B.Cu")
+		(net "/04_PPG/PPG2_PD2_IN")
+	)
+	(segment
+		(start 98.05 101.2)
+		(end 91.5 101.2)
 		(width 0.1)
 		(layer "B.Cu")
@@
 	)
 	(segment
-		(start 90.2 98.7)
-		(end 90.2 94.5)
+		(start 90.2 96.4)
+		(end 90.2 98.7)
 		(width 0.1)
 		(layer "B.Cu")
@@
 	(segment
 		(start 92.1 98.7)
-		(end 90.2 98.7)
+		(end 92.1 98.4)
 		(width 0.1)
 		(layer "B.Cu")
@@
 	)
 	(segment
-		(start 97 96.4)
-		(end 90.2 96.4)
+		(start 90.2 96.4)
+		(end 90.2 94.5)
 		(width 0.1)
 		(layer "B.Cu")
@@
 	(segment
 		(start 98.05 100)
-		(end 97 96.4)
+		(end 98.05 101.2)
+		(width 0.1)
+		(layer "B.Cu")
+		(net "/04_PPG/PPG2_PD_GND")
+	)
+	(segment
+		(start 99.15 96.4)
+		(end 90.2 96.4)
+		(width 0.1)
+		(layer "B.Cu")
+		(net "/04_PPG/PPG2_PD_GND")
+	)
+	(segment
+		(start 100 95.55)
+		(end 99.15 96.4)
+		(width 0.1)
+		(layer "B.Cu")
+		(net "/04_PPG/PPG2_PD_GND")
+	)
+	(segment
+		(start 90.2 98.7)
+		(end 92.1 98.7)
+		(width 0.1)
+		(layer "B.Cu")
+		(net "/04_PPG/PPG2_PD_GND")
+	)
+	(segment
+		(start 91.5 101.2)
+		(end 91.5 98.7)
+		(width 0.1)
+		(layer "B.Cu")
+		(net "/04_PPG/PPG2_PD_GND")
+	)
+	(segment
+		(start 91.5 98.7)
+		(end 92.1 98.7)
 		(width 0.1)
 		(layer "B.Cu")
@@
 	)
 	(segment
-		(start 94.5 100)
-		(end 93.5 99)
+		(start 92.5 98.5)
+		(end 92.5 98.4)
 		(width 0.1)
 		(layer "B.Cu")
@@
 	)
 	(segment
-		(start 92.5 98.5)
-		(end 92.5 98.4)
+		(start 93.5 99)
+		(end 92.5 98.5)
 		(width 0.1)
 		(layer "B.Cu")
@@
 	)
 	(segment
-		(start 95.55 100)
-		(end 94.5 100)
+		(start 94.5 100)
+		(end 93.5 99)
 		(width 0.1)
 		(layer "B.Cu")
@@
 	)
 	(segment
-		(start 93.5 99)
-		(end 92.5 98.5)
+		(start 95.55 100)
+		(end 94.5 100)
 		(width 0.1)
 		(layer "B.Cu")

Commit message: fix(pcb): foundation correction round 4 closure
- Y101: select Abracon ABS06-32.768KHZ-6-1-T (2012-class SMD crystal) matching 2012 footprint
- Y101/C118/C119: rotate Y101 180 deg to align XO32 West and XI32 East; uncrossed planar routing
- Parity: synchronize C118, C119, Y101, Y102, Y1 values between schematic and PCB (0 mismatches)
- PPG guards: close NT401.2 and NT402.2 to In6.Cu GND plane via B.Cu microvias (4 channels complete)
- Rules: reconcile HighSpeed_50R track_width to 0.100 mm in .kicad_pro; refine *1V8* to *VOUT*1V8*
- GNSS: update note to cite MAX-F10S Integration Manual UBXDOC-963802114-12892 R01 and south RF_IN
Parts:
- C118, C119: value TBD <=10pF -> 8.2pF
- Y1: value 40MHz_CL8pF_ESR100R_1612 -> NX1612SA-40M-EXS00A-CS14264
- Y101: value 32.768kHz / low-CL TBD -> ABS06-32.768KHZ-6-1-T
- Y102: value 48MHz / CL=8-11pF / ESR<=60R -> NX1612SA-48M-EXS00A-CS14265
- moved C118 5.20 mm to (101.6, 93.3)
- moved C119 5.20 mm to (96.4, 93.3), turned to 180 degrees
- turned Y101 to 180 degrees
Routing:
- net GND: track 0.00 -> 0.70 mm, vias 0 -> 2
Changed lines of the file:
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@@
 	(footprint "Crystal:Crystal_SMD_2012-2Pin_2.0x1.2mm"
 		(layer "F.Cu")
-		(at 99 93.3)
+		(at 99 93.3 180)
 		(descr "2012/2, Crystal, 2.0x1.2mm package, SMD, http://txccrystal.com/images/pdf/9ht11.pdf")
 		(property "Reference" "Y101"
-			(at 0 -1.8 0)
+			(at 0 -1.8 180)
 			(layer "F.SilkS")
 			(effects
@@
 			)
 		)
-		(property "Value" "32.768kHz / low-CL TBD"
-			(at 0 1.8 0)
+		(property "Value" "ABS06-32.768KHZ-6-1-T"
+			(at 0 1.8 180)
 			(layer "F.Fab")
 			(effects
@@
 			)
 		)
-		(property "Description" "32.768kHz RTC crystal; choose CL compatible with <=10pF external cap per pin"
+		(property "Description" "32.768kHz RTC crystal; 6pF CL, 90k ESR, 2012 package compatible with Apollo510B"
 			(at 0 0 0)
 			(layer "F.Fab")
@@
 			)
 		)
-		(property "Value" "40MHz_CL8pF_ESR100R_1612"
+		(property "Value" "NX1612SA-40M-EXS00A-CS14264"
 			(at 0 1.6 0)
 			(layer "F.Fab")
@@
 			)
 		)
-		(property "Value" "48MHz / CL=8-11pF / ESR<=60R"
+		(property "Value" "NX1612SA-48M-EXS00A-CS14265"
 			(at 0 1.6 270)
 			(layer "F.Fab")
@@
 	(footprint "Capacitor_SMD:C_0201_0603Metric"
 		(layer "F.Cu")
-		(at 101.6 93.3)
+		(at 96.4 93.3 180)
 		(descr "Capacitor SMD 0201 (0603 Metric), square (rectangular) end terminal, IPC-7351 nominal, (Body size source: https://www.vishay.com/docs/20052/crcw0201e3.pdf)")
 		(tags "capacitor")
 		(property "Reference" "C119"
-			(at 0 -1.05 0)
+			(at 0 -1.05 180)
 			(layer "F.SilkS")
 			(effects
@@
 			)
 		)
-		(property "Value" "TBD <=10pF"
-			(at 0 1.05 0)
+		(property "Value" "8.2pF"
+			(at 0 1.05 180)
 			(layer "F.Fab")
 			(effects
@@
 	(footprint "Capacitor_SMD:C_0201_0603Metric"
 		(layer "F.Cu")
-		(at 96.4 93.3)
+		(at 101.6 93.3)
 		(descr "Capacitor SMD 0201 (0603 Metric), square (rectangular) end terminal, IPC-7351 nominal, (Body size source: https://www.vishay.com/docs/20052/crcw0201e3.pdf)")
 		(tags "capacitor")
@@
 			)
 		)
-		(property "Value" "TBD <=10pF"
+		(property "Value" "8.2pF"
 			(at 0 1.05 0)
 			(layer "F.Fab")
@@
 		(net "/04_PPG/PPG2_PD1_IN")
 	)
+	(segment
+		(start 102.3 108.5)
+		(end 102.7 108.5)
+		(width 0.1)
+		(layer "B.Cu")
+		(net "GND")
+	)
+	(via micro
+		(at 102.7 108.5)
+		(size 0.22)
+		(drill 0.1)
+		(layers "In6.Cu" "B.Cu")
+		(net "GND")
+	)
+	(segment
+		(start 92.4 94.5)
+		(end 92.7 94.5)
+		(width 0.1)
+		(layer "B.Cu")
+		(net "GND")
+	)
+	(via micro
+		(at 92.7 94.5)
+		(size 0.22)
+		(drill 0.1)
+		(layers "In6.Cu" "B.Cu")
+		(net "GND")
+	)
 	(zone

Commit message: fix(pcb): foundation correction round 5 closure
Parts:
- Y101: footprint Crystal:Crystal_SMD_2012-2Pin_2.0x1.2mm -> sportwatch_custom:Crystal_SMD_ABS06_2.0x1.2mm
Changed lines of the file:
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@@
 		)
 	)
-	(footprint "Crystal:Crystal_SMD_2012-2Pin_2.0x1.2mm"
+	(footprint "sportwatch_custom:Crystal_SMD_ABS06_2.0x1.2mm"
 		(layer "F.Cu")
 		(at 99 93.3 180)
-		(descr "2012/2, Crystal, 2.0x1.2mm package, SMD, http://txccrystal.com/images/pdf/9ht11.pdf")
+		(descr "Abracon ABS06 32.768kHz SMD crystal, 2.0x1.2x0.6mm body, 2-pin nonpolar. Recommended land pattern: 0.75x1.4mm lands, 0.7mm inner gap, 1.45mm centers (Abracon datasheet rev 11-23-20)")
 		(property "Reference" "Y101"
-			(at 0 -1.8 180)
+			(at 0 -1.6 180)
 			(layer "F.SilkS")
 			(effects
 				(font
-					(size 1 1)
-					(thickness 0.15)
+					(size 0.8 0.8)
+					(thickness 0.12)
 				)
 			)
 		)
 		(property "Value" "ABS06-32.768KHZ-6-1-T"
-			(at 0 1.8 180)
+			(at 0 1.6 180)
 			(layer "F.Fab")
 			(effects
 				(font
-					(size 1 1)
-					(thickness 0.15)
+					(size 0.8 0.8)
+					(thickness 0.12)
 				)
 			)
@@
 			)
 		)
-		(property "KiLib_Generator" "crystal_resonator_oscillator"
-			(at 0 0 0)
-			(layer "F.SilkS")
-			(hide yes)
-			(effects
-				(font
-					(size 1 1)
-					(thickness 0.15)
-				)
-			)
-		)
 		(sheetname "/01_APOLLO510B/")
 		(sheetfile "01_APOLLO510B.kicad_sch")
@@
 		(duplicate_pad_numbers_are_jumpers no)
 		(fp_line
-			(start -1.26 -0.86)
-			(end -1.26 0.86)
+			(start -1.25 0.4)
+			(end -1.25 0.7)
 			(stroke
 				(width 0.12)
@@
 		)
 		(fp_line
-			(start -1.26 0.86)
-			(end 1.26 0.86)
+			(start -0.2 0.85)
+			(end 0.2 0.85)
 			(stroke
 				(width 0.12)
@@
 		)
 		(fp_line
-			(start 1.26 -0.86)
-			(end -1.26 -0.86)
+			(start -0.2 -0.85)
+			(end 0.2 -0.85)
 			(stroke
 				(width 0.12)
@@
 			(layer "F.SilkS")
 		)
-		(fp_circle
-			(center 0 0)
-			(end 0.2 0)
-			(stroke
-				(width 0.1)
-				(type solid)
-			)
-			(fill yes)
-			(layer "F.Adhes")
-		)
 		(fp_rect
-			(start -1.5 -1.1)
-			(end 1.5 1.1)
+			(start -1.35 -0.95)
+			(end 1.35 0.95)
 			(stroke
 				(width 0.05)
@@
 			(effects
 				(font
-					(size 0.5 0.5)
-					(thickness 0.08)
+					(size 0.4 0.4)
+					(thickness 0.06)
 				)
 			)
 		)
 		(pad "1" smd roundrect
-			(at -0.7 0)
-			(size 0.6 1.1)
+			(at -0.725 0)
+			(size 0.75 1.4)
 			(layers "F.Cu" "F.Mask" "F.Paste")
 			(roundrect_rratio 0.25)
@@
 		)
 		(pad "2" smd roundrect
-			(at 0.7 0)
-			(size 0.6 1.1)
+			(at 0.725 0)
+			(size 0.75 1.4)
 			(layers "F.Cu" "F.Mask" "F.Paste")
 			(roundrect_rratio 0.25)

Commit message: pcb: complete Rev-A multi-board placement Phase 1
Parts:
- removed C403, C404, C405, C406, C407, C408, C4102, C4202, C802: 100nF, Capacitor_SMD:C_0402_1005Metric
- removed C4101, C4201: 22uF, Capacitor_SMD:C_0402_1005Metric
- removed C4103, C4203: 1.0uF, Capacitor_SMD:C_0402_1005Metric
- removed C4104, C4204: 10uF, Capacitor_SMD:C_0402_1005Metric
- removed D401, D402, D403, D404: SFH7018A Q65113A6157, sportwatch_custom:OSRAM_SFH7018A_2.4x2.4mm
- removed D405, D406, D407: SFH4053B Q65115A1586, sportwatch_custom:OSRAM_SFH4053B_1.0x0.5mm
- removed D413, D414, D423, D424: SFH2703H Q65115A2199, sportwatch_custom:OSRAM_SFH2703_3.2x2.0mm
- removed NT401: PPG1_PD_GND_TIE, NetTie:NetTie-2_SMD_Pad0.5mm
- removed NT402: PPG2_PD_GND_TIE, NetTie:NetTie-2_SMD_Pad0.5mm
- removed R401, R402, R405: 100k, Resistor_SMD:R_0402_1005Metric
- removed R403, R404: 47k, Resistor_SMD:R_0402_1005Metric
- removed R408, R409: 10k, Resistor_SMD:R_0402_1005Metric
- removed U12, U13: MAX86141ENP+T, sportwatch_custom:21-100134_N201A2-1_MXM
- removed U402, U403, U404, U405, U406, U407: TS5A12301E, Package_BGA:Texas_DSBGA-6_0.76x1.16mm_Layout2x3_P0.4mm
- removed U6: MAX30208CLB+T, sportwatch_custom:21-100265_MXM
- C206, C901, C902, C903, C904, C905, C906, R901, R902, R903, R904, R905, R906, R907, R908, R909, R910: moved to B.Cu
- moved R110 187.6 mm to (91.8, 117.2), turned to 90 degrees
- moved R107 184.1 mm to (84.8, 108.0)
- moved R106 180.2 mm to (99.5, 101.3)
- moved R104 180.1 mm to (82.5, 108.0)
- moved R109 180.0 mm to (80.2, 108.0)
- moved R108 177.0 mm to (92.8, 102.5)
- moved C701 175.0 mm to (109.2, 95.9)
- moved R101 173.5 mm to (105.2, 93.5), turned to 90 degrees
- moved C702 172.8 mm to (107.0, 95.9)
- moved R105 172.4 mm to (97.3, 101.3)
- moved J1301 172.2 mm to (107.0, 114.0)
- moved U105 171.7 mm to (87.5, 100.8)
- moved C703 171.3 mm to (111.5, 95.9)
- moved U702 170.4 mm to (109.2, 93.2)
- moved C121 170.3 mm to (84.8, 92.0)
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Connections:
- net /02_POWER/VBUSIN renamed VBUSIN
- net /04_PPG/PPG_VLED renamed PPG_VLED
- net /ALS_INT renamed ALS_INT
- net /BARO_INT renamed BARO_INT
- net /ENV_I2C_SCL renamed ENV_I2C_SCL
- net /ENV_I2C_SDA renamed ENV_I2C_SDA
- net /VBAT renamed VBAT
- net /VOUT1_1V8 renamed VOUT1_1V8
- U101 pad C8: /PPG2_INT_N -> PPG2_INT_N
- U101 pad D8: /PPG1_INT_N -> PPG1_INT_N
- U101 pad D9: /PPG1_CS_N -> PPG1_CS_N
- U101 pad H13: /PPG_SAMPLE_SYNC -> PPG_SAMPLE_SYNC
- U101 pad K5: /PPG_SPI_SCLK -> PPG_SPI_SCLK
- U101 pad L5: /PPG_SPI_MOSI -> PPG_SPI_MOSI
- U101 pad L7: /PPG_SPI_MISO -> PPG_SPI_MISO
- U101 pad M5: /PPG2_CS_N -> PPG2_CS_N
Routing:
- net /04_PPG/PPG2_PD_GND: track 28.6 -> 0.00 mm
- net /04_PPG/PPG1_PD_GND: track 19.3 -> 0.00 mm
- net /04_PPG/PPG2_PD2_IN: track 7.50 -> 0.00 mm
- net /04_PPG/PPG1_PD1_IN: track 6.68 -> 0.00 mm
- net /04_PPG/PPG2_PD1_IN: track 3.68 -> 0.00 mm
- net /04_PPG/PPG1_PD2_IN: track 1.92 -> 0.00 mm
- net GND: track 0.70 -> 0.00 mm, vias 2 -> 0
Other:
- board text added: "B.Cu CLEARANCE POCKETS REQUIRED / HEIGHT + INSULATION + PACK TOLERANCE TBD"
- board text added: "BATTERY WIRE EXIT"
- board text added: "BLE radiator opportunity"
- board text added: "DEVELOPMENT ENVELOPE D46 / NOT FINAL EDGE.CUTS F.Cu = DISPLAY / B.Cu = BATTERY LRA lower-level SOUTH pocket / no same-Z battery overlap approval"
- board text added: "GNSS radiator / feed opportunity"
- board text added: "J1501 sensor FPC"
- board text added: "J201 / BODY TBD"
- board text added: "LPR454440 - NOMINAL BATTERY PROJECTION ONLY D44.0 x 4.5 mm / FINAL PROTECTED PACK ENVELOPE TBD"
- board text added: "SHIELD-READY DIGITAL CORE (U101 SoC) - STEPPED PERIMETER / NO COURTYARD CROSSINGS / CONTACTS TBD"
- board text added: "Wi-Fi radiator opportunity"
- board text added: "main charger protection / J202"
- board text added: "support search SE"
- board text added: "support search SW"
- board text added: "support search north-east"
