File: rear_sensor/08_TEMPERATURE.kicad_sch (KiCad schematic)
At the start: 8 parts, among them U4 BMP585, U5 OPT4001DTSR

Commit message: foundation correction
Parts:
- removed C801, C803, C804: 100nF, Capacitor_SMD:C_0402_1005Metric, symbol Device:C
- removed R801, R802: 4.7k, Resistor_SMD:R_0402_1005Metric, symbol Device:R
- removed R803: 10k, Resistor_SMD:R_0402_1005Metric, symbol Device:R
- removed U4: BMP585, sportwatch_custom:LGA9_BMP585_BOS, symbol 2026-09-16_05-56-22:BMP585
- removed U5: OPT4001DTSR, sportwatch_custom:DTS0008A-MFG, symbol 2026-09-16_05-59-08:OPT4001DTSR
- added C802: 100nF, Capacitor_SMD:C_0402_1005Metric, symbol Device:C
- added U6: MAX30208CLB+T, sportwatch_custom:21-100265_MXM, symbol 2026-09-16_05-57-26:MAX30208CLB+T
Connections:
- net ENV_I2C_SCL: now also U6.9 (SCL)
- net ENV_I2C_SDA: now also U6.8 (SDA)
- net GND: now also C802.2, U6.10 (GPIO0), U6.4 (GND), U6.5 (GND), U6.6 (GND), U6.7 (GPIO1)
- net VOUT1_1V8: now also C802.1, U6.1 (VDD), U6.2 (VDD), U6.3 (VDD)
- no-connect marks 3 -> 0
Other:
- note added: "U6.7/U6.10 grounded. No temperature IRQ. Thermal island requires later mechanical review."
- note removed: "MAX30208 U6/C802 moved to REAR. R801/R802 remain MAIN; no duplicated rear pull-ups."
- title: MAIN - BMP585 / OPT4001 / ENV I2C pull-ups -> REAR - MAX30208 ten-pin Thin LGA / polled temperature
